Commit message: description: remove Gazebo material defs
We now have Collada files with the right colors

Signed-off-by: Wolfgang Wiedmeyer <wolfgang.wiedmeyer@kit.edu>

File: rll_description/urdf/iiwa7/iiwa.gazebo.xacro (robot description, xacro)
@@ -10,5 +10,4 @@
     <!-- Link0 -->
     <gazebo reference="${robot_name}_link_0">
-      <material>Gazebo/Grey</material>
       <mu1>0.2</mu1>
       <mu2>0.2</mu2>
@@ -16,5 +15,4 @@
     <!-- Link1 -->
     <gazebo reference="${robot_name}_link_1">
-      <material>Gazebo/Orange</material>
       <mu1>0.2</mu1>
       <mu2>0.2</mu2>
@@ -22,5 +20,4 @@
     <!-- Link2 -->
     <gazebo reference="${robot_name}_link_2">
-      <material>Gazebo/Orange</material>
       <mu1>0.2</mu1>
       <mu2>0.2</mu2>
@@ -28,5 +25,4 @@
     <!-- Link3 -->
     <gazebo reference="${robot_name}_link_3">
-      <material>Gazebo/Orange</material>
       <mu1>0.2</mu1>
       <mu2>0.2</mu2>
@@ -34,5 +30,4 @@
     <!-- Link4 -->
     <gazebo reference="${robot_name}_link_4">
-      <material>Gazebo/Orange</material>
       <mu1>0.2</mu1>
       <mu2>0.2</mu2>
@@ -40,5 +35,4 @@
     <!-- Link5 -->
     <gazebo reference="${robot_name}_link_5">
-      <material>Gazebo/Orange</material>
       <mu1>0.2</mu1>
       <mu2>0.2</mu2>
@@ -46,5 +40,4 @@
     <!-- Link6 -->
     <gazebo reference="${robot_name}_link_6">
-      <material>Gazebo/Orange</material>
       <mu1>0.2</mu1>
       <mu2>0.2</mu2>
@@ -52,5 +45,4 @@
     <!-- Link7 -->
     <gazebo reference="${robot_name}_link_7">
-      <material>Gazebo/Grey</material>
       <mu1>0.2</mu1>
       <mu2>0.2</mu2>
