Commit message: description: remove unneeded utilities for iiwa
Signed-off-by: Wolfgang Wiedmeyer <wolfgang.wiedmeyer@kit.edu>

File: rll_description/urdf/iiwa7/iiwa7.xacro (robot description, xacro)
@@ -5,6 +5,4 @@
   <!-- Import Transmissions -->
   <xacro:include filename="$(find rll_description)/urdf/iiwa7/iiwa.transmission.xacro" />
-  <!-- Include Utilities -->
-  <xacro:include filename="$(find rll_description)/urdf/iiwa7/utilities.xacro" />
   <!-- some constants -->
   <xacro:property name="safety_controller_k_pos" value="100" />
@@ -13,4 +11,5 @@
   <xacro:property name="max_effort" value="300"/>
   <xacro:property name="max_velocity" value="10"/>
+  <xacro:property name="PI" value="3.1415926535897931"/>
   <xacro:macro name="iiwa7" params="parent hardware_interface robot_name *origin">
     <!--joint between {parent} and link_0-->

Commit message: Corrected the moments of inertia of the links on iiwa7. Added a camera to the world file for future recording

File: rll_description/urdf/iiwa7/iiwa7.xacro (robot description, xacro)
@@ -20,5 +20,5 @@
     <link name="${robot_name}_link_0">
       <inertial>
-        <origin xyz="-0.1 0 0.07" rpy="0 0 0"/>
+        <origin xyz="-0.01 0 0.07" rpy="0 0 0"/>
         <mass value="5"/>
         <inertia ixx="0.05"  ixy="0"  ixz="0" iyy="0.06" iyz="0" izz="0.03" />
@@ -59,5 +59,5 @@
         <origin xyz="0 -0.03 0.12" rpy="0 0 0"/>
         <mass value="3.4525"/>
-        <inertia ixx="0.02183"  ixy="0"  ixz="0" iyy="0.007703" iyz="-0.003887" izz="0.02083" />
+        <inertia ixx="0.02183"  ixy="0"  ixz="0" iyy="0.02081" iyz="0.003883" izz="0.007697" />
       </inertial>
       <visual>
@@ -87,7 +87,7 @@
     <link name="${robot_name}_link_2">
       <inertial>
-        <origin xyz="0.0003 0.059 0.042" rpy="0 0 0"/>
+        <origin xyz="0.000 0.034417 0.0673286" rpy="0 0 0"/>
         <mass value="3.4821"/>
-        <inertia ixx="0.02076"  ixy="0"  ixz="-0.003626" iyy="0.02179" iyz="0" izz="0.00779" />
+        <inertia ixx="0.02177"  ixy="0"  ixz="0.00" iyy="0.02075" iyz="0.003621" izz="0.00779" />
       </inertial>
       <visual>
@@ -117,7 +117,7 @@
     <link name="${robot_name}_link_3">
       <inertial>
-        <origin xyz="0 0.03 0.13" rpy="0 0 0"/>
+        <origin xyz="0 0.0295 0.1258" rpy="0 0 0"/>
         <mass value="4.05623"/>
-        <inertia ixx="0.03204"  ixy="0"  ixz="0" iyy="0.00972" iyz="0.006227" izz="0.03042" />
+        <inertia ixx="0.03204"  ixy="0"  ixz="0" iyy="0.03044" iyz="-0.006231" izz="0.009726" />
       </inertial>
       <visual>
@@ -147,7 +147,7 @@
     <link name="${robot_name}_link_4">
       <inertial>
-        <origin xyz="0 0.067 0.034" rpy="0 0 0"/>
+        <origin xyz="0 -0.034 0.067" rpy="0 0 0"/>
         <mass value="3.4822"/>
-        <inertia ixx="0.02178"  ixy="0"  ixz="0" iyy="0.02075" iyz="-0.003625" izz="0.007785" />
+        <inertia ixx="0.021775"  ixy="0"  ixz="0" iyy="0.02075" iyz="-0.003621" izz="0.007783" />
       </inertial>
       <visual>
@@ -177,7 +177,7 @@
     <link name="${robot_name}_link_5">
       <inertial>
-        <origin xyz="0.0001 0.021 0.076" rpy="0 0 0"/>
+        <origin xyz="0.0001 -0.02263 -0.1365" rpy="0 0 0"/>
         <mass value="2.1633"/>
-        <inertia ixx="0.01287"  ixy="0"  ixz="0" iyy="0.005708" iyz="-0.003946" izz="0.01112" />
+        <inertia ixx="0.01287"  ixy="0"  ixz="0" iyy="0.01112" iyz="0.003943" izz="0.0057128" />
       </inertial>
       <visual>
@@ -207,7 +207,7 @@
     <link name="${robot_name}_link_6">
       <inertial>
-        <origin xyz="0 0.0006 0.0004" rpy="0 0 0"/>
+        <origin xyz="0 0.00047 0.002124" rpy="0 0 0"/>
         <mass value="2.3466"/>
-        <inertia ixx="0.006509"  ixy="0"  ixz="0" iyy="0.006259" iyz="0.00031891" izz="0.004527" />
+        <inertia ixx="0.006522"  ixy="0"  ixz="0" iyy="0.006270" iyz="0.00032280" izz="0.0045345" />
       </inertial>
       <visual>
@@ -237,7 +237,7 @@
     <link name="${robot_name}_link_7">
       <inertial>
-        <origin xyz="0 0 0.02" rpy="0 0 0"/>
+        <origin xyz="0 0 0.1" rpy="0 0 0"/>
         <mass value="3.129"/>
-        <inertia ixx="0.01464"  ixy="0.0005912"  ixz="0" iyy="0.01465" iyz="0" izz="0.002872" />
+        <inertia ixx="0.0022711"  ixy="0.0000221"  ixz="0" iyy="0.0022807" iyz="0" izz="0.002872" />
       </inertial>
       <visual>

File: rll_description/urdf/rll.gazebo.xacro (robot description, xacro)
@@ -8,5 +8,5 @@
       <kp>1000000.0</kp>
       <kd>1.0</kd>
-      <fdir1>0 0 1</fdir1>
+      <fdir1>1 0 0</fdir1>
       <minDepth>0.001</minDepth>
       <!-- <static>true</static> -->

Commit message: description: set pos limits according to Sunrise safety config
Signed-off-by: Wolfgang Wiedmeyer <wolfgang.wiedmeyer@kit.edu>

File: rll_description/urdf/iiwa7/iiwa7.xacro (robot description, xacro)
@@ -47,8 +47,8 @@
       <origin xyz="0 0 0.157" rpy="0 0 0"/>
       <axis xyz="0 0 1"/>
-      <limit lower="${-170 * pi / 180}" upper="${170 * pi / 180}"
+      <limit lower="${-169 * pi / 180}" upper="${169 * pi / 180}"
              effort="${max_effort}" velocity="${98 * pi / 180}" />
-      <safety_controller soft_lower_limit="${-168 * pi / 180}"
-                         soft_upper_limit="${168 * pi / 180}"
+      <safety_controller soft_lower_limit="${-167 * pi / 180}"
+                         soft_upper_limit="${167 * pi / 180}"
                          k_position="${safety_controller_k_pos}"
                          k_velocity="${safety_controller_k_vel}"/>
@@ -77,8 +77,8 @@
       <origin xyz="0 0 0.183" rpy="0 0 0"/>
       <axis xyz="0 1 0"/>
-      <limit lower="${-120 * pi / 180}" upper="${120 * pi / 180}"
+      <limit lower="${-119 * pi / 180}" upper="${119 * pi / 180}"
              effort="${max_effort}" velocity="${98 * pi / 180}" />
-      <safety_controller soft_lower_limit="${-118 * pi / 180}"
-                         soft_upper_limit="${118 * pi / 180}"
+      <safety_controller soft_lower_limit="${-117 * pi / 180}"
+                         soft_upper_limit="${117 * pi / 180}"
                          k_position="${safety_controller_k_pos}"
                          k_velocity="${safety_controller_k_vel}"/>
@@ -107,8 +107,8 @@
       <origin xyz="0 0 0.185" rpy="0 0 0"/>
       <axis xyz="0 0 1"/>
-      <limit lower="${-170 * pi / 180}" upper="${170 * pi / 180}"
+      <limit lower="${-169 * pi / 180}" upper="${169 * pi / 180}"
              effort="${max_effort}" velocity="${100 * pi / 180}" />
-      <safety_controller soft_lower_limit="${-168 * pi / 180}"
-                         soft_upper_limit="${168 * pi / 180}"
+      <safety_controller soft_lower_limit="${-167 * pi / 180}"
+                         soft_upper_limit="${167 * pi / 180}"
                          k_position="${safety_controller_k_pos}"
                          k_velocity="${safety_controller_k_vel}"/>
@@ -137,8 +137,8 @@
       <origin xyz="0 0 0.215" rpy="0 0 0"/>
       <axis xyz="0 -1 0"/>
-      <limit lower="${-120 * pi / 180}" upper="${120 * pi / 180}"
+      <limit lower="${-119 * pi / 180}" upper="${119 * pi / 180}"
              effort="${max_effort}" velocity="${130 * pi / 180}" />
-      <safety_controller soft_lower_limit="${-118 * pi / 180}"
-                         soft_upper_limit="${118 * pi / 180}"
+      <safety_controller soft_lower_limit="${-117 * pi / 180}"
+                         soft_upper_limit="${117 * pi / 180}"
                          k_position="${safety_controller_k_pos}"
                          k_velocity="${safety_controller_k_vel}"/>
@@ -167,8 +167,8 @@
       <origin xyz="0 0 0.4" rpy="0 0 0"/>
       <axis xyz="0 0 1"/>
-      <limit lower="${-170 * pi / 180}" upper="${170 * pi / 180}"
+      <limit lower="${-169 * pi / 180}" upper="${169 * pi / 180}"
              effort="${max_effort}" velocity="${140 * pi / 180}" />
-      <safety_controller soft_lower_limit="${-168 * pi / 180}"
-                         soft_upper_limit="${168 * pi / 180}"
+      <safety_controller soft_lower_limit="${-167 * pi / 180}"
+                         soft_upper_limit="${167 * pi / 180}"
                          k_position="${safety_controller_k_pos}"
                          k_velocity="${safety_controller_k_vel}"/>
@@ -197,8 +197,8 @@
       <origin xyz="0 0 0" rpy="0 0 0"/>
       <axis xyz="0 1 0"/>
-      <limit lower="${-120 * pi / 180}" upper="${120 * pi / 180}"
+      <limit lower="${-119 * pi / 180}" upper="${119 * pi / 180}"
              effort="${max_effort}" velocity="${180 * pi / 180}" />
-      <safety_controller soft_lower_limit="${-118 * pi / 180}"
-                         soft_upper_limit="${118 * pi / 180}"
+      <safety_controller soft_lower_limit="${-117 * pi / 180}"
+                         soft_upper_limit="${117 * pi / 180}"
                          k_position="${safety_controller_k_pos}"
                          k_velocity="${safety_controller_k_vel}"/>
@@ -227,8 +227,8 @@
       <origin xyz="0 0 0" rpy="0 0 0"/>
       <axis xyz="0 0 1"/>
-      <limit lower="${-175 * pi / 180}" upper="${175 * pi / 180}"
+      <limit lower="${-174 * pi / 180}" upper="${174 * pi / 180}"
              effort="${max_effort}" velocity="${180 * pi / 180}" />
-      <safety_controller soft_lower_limit="${-173 * pi / 180}"
-                         soft_upper_limit="${173 * pi / 180}"
+      <safety_controller soft_lower_limit="${-172 * pi / 180}"
+                         soft_upper_limit="${172 * pi / 180}"
                          k_position="${safety_controller_k_pos}"
                          k_velocity="${safety_controller_k_vel}"/>

Commit message: description: remove unused max_velocity parameter
Signed-off-by: Wolfgang Wiedmeyer <wolfgang.wiedmeyer@kit.edu>

File: rll_description/urdf/iiwa7/iiwa7.xacro (robot description, xacro)
@@ -9,6 +9,6 @@
   <xacro:property name="safety_controller_k_vel" value="2" />
   <xacro:property name="joint_damping" value="0.5" />
+  <!-- TODO: set the correct individual effort values for every joint -->
   <xacro:property name="max_effort" value="300"/>
-  <xacro:property name="max_velocity" value="10"/>
   <xacro:macro name="iiwa7" params="parent hardware_interface robot_name *origin">
     <!--joint between {parent} and link_0-->
