Commit message: description: use a simplified collision model for iiwa
The model is similar to the collision model of the Sunrise controller
which exclusively uses spheres. The Sunrise controller model is detailed in
the Sunrise OS docs.
However the Sunrise controller model does not cover the whole robot. Parts
of link 1, 3 and 5 are not covered by the small spheres.
To overcome this limitation, cylinders are used for these three links. The
cylinder dimensions were chosen to cover the whole link while not being
smaller than the spheres from the Sunrise model at any point.

This new collision model should make it easier to be compatible with the
Sunrise model and to avoid discrepancies between the two when running
trajectories on the real robot.
The model also leads to faster collision checking in Moveit and reduces
CPU load in Gazebo. The accuracy of the model should still be sufficient
for our use cases and it should not limit motions that were previously
possible.

Signed-off-by: Wolfgang Wiedmeyer <wolfgang.wiedmeyer@kit.edu>

File: rll_description/urdf/iiwa7/iiwa7.xacro (robot description, xacro)
@@ -25,14 +25,9 @@
       </visual>
       <collision>
-        <geometry>
-          <mesh filename="package://rll_description/meshes/iiwa7/collision/base.stl"/>
-        </geometry>
-      </collision>
-      <self_collision_checking>
-        <origin xyz="0 0 0" rpy="0 0 0"/>
-        <geometry>
-          <capsule radius="0.15" length="0.25"/>
-        </geometry>
-      </self_collision_checking>
+	<origin xyz="0 0 0.0785"/>
+        <geometry>
+	  <cylinder length="0.157" radius="0.135"/>
+        </geometry>
+      </collision>
     </link>
     <!-- joint between link_0 and link_1 -->
@@ -62,6 +57,7 @@
       </visual>
       <collision>
-        <geometry>
-          <mesh filename="package://rll_description/meshes/iiwa7/collision/link1.stl"/>
+	<origin xyz="0 -0.01 0.06"/>
+        <geometry>
+	  <cylinder length="0.12" radius="0.1"/>
         </geometry>
       </collision>
@@ -92,6 +88,7 @@
       </visual>
       <collision>
-        <geometry>
-          <mesh filename="package://rll_description/meshes/iiwa7/collision/link2.stl"/>
+	<origin xyz="0 0 0"/>
+        <geometry>
+	  <sphere radius="0.125"/>
         </geometry>
       </collision>
@@ -122,6 +119,7 @@
       </visual>
       <collision>
-        <geometry>
-          <mesh filename="package://rll_description/meshes/iiwa7/collision/link3.stl"/>
+	<origin xyz="0 0.01 0.02"/>
+        <geometry>
+	  <cylinder length="0.28" radius="0.1"/>
         </geometry>
       </collision>
@@ -152,6 +150,7 @@
       </visual>
       <collision>
-        <geometry>
-          <mesh filename="package://rll_description/meshes/iiwa7/collision/link4.stl"/>
+	<origin xyz="0 0 0"/>
+        <geometry>
+	  <sphere radius="0.125"/>
         </geometry>
       </collision>
@@ -182,6 +181,7 @@
       </visual>
       <collision>
-        <geometry>
-          <mesh filename="package://rll_description/meshes/iiwa7/collision/link5.stl"/>
+	<origin xyz="0 -0.01 -0.18"/>
+        <geometry>
+	  <cylinder length="0.3" radius="0.1"/>
         </geometry>
       </collision>
@@ -212,6 +212,7 @@
       </visual>
       <collision>
-        <geometry>
-          <mesh filename="package://rll_description/meshes/iiwa7/collision/link6.stl"/>
+	<origin xyz="0 -0.03 0"/>
+        <geometry>
+	  <sphere radius="0.08"/>
         </geometry>
       </collision>
@@ -242,6 +243,7 @@
       </visual>
       <collision>
-        <geometry>
-          <mesh filename="package://rll_description/meshes/iiwa7/collision/link7.stl"/>
+	<origin xyz="0 0 -0.01"/>
+        <geometry>
+	  <sphere radius="0.085"/>
         </geometry>
       </collision>
@@ -253,4 +255,10 @@
     </joint>
     <link name="${robot_name}_link_ee">
+      <collision>
+	<origin xyz="0 0 -0.046"/>
+        <geometry>
+	  <sphere radius="0.065"/>
+        </geometry>
+      </collision>
     </link>
     <xacro:iiwa_gazebo robot_name="${robot_name}" />

File: rll_moveit_config/config/rll_cell.xacro (robot description, xacro)
@@ -67,4 +67,5 @@
     <disable_collisions link1="axis_cam_base" link2="$(arg robot_name)_link_6" reason="Never" />
     <disable_collisions link1="axis_cam_base" link2="$(arg robot_name)_link_7" reason="Never" />
+    <disable_collisions link1="axis_cam_base" link2="$(arg robot_name)_link_ee" reason="Never" />
     <disable_collisions link1="axis_cam_base" link2="$(arg robot_name)_roboception_adapter" reason="Never" />
     <disable_collisions link1="axis_cam_base" link2="$(arg robot_name)_roboception_camera_uncal" reason="Never" />
@@ -73,5 +74,5 @@
     <disable_collisions link1="axis_cam_base" link2="table" reason="Never" />
     <disable_collisions link1="axis_cam_base" link2="wall_back" reason="Never" />
-    <disable_collisions link1="axis_cam_base" link2="wall_front" reason="Never" />
+    <disable_collisions link1="axis_cam_base" link2="wall_front" reason="Default" />
     <disable_collisions link1="axis_cam_base" link2="wall_left" reason="Never" />
     <disable_collisions link1="axis_cam_base" link2="wall_right" reason="Default" />
@@ -91,4 +92,5 @@
     <disable_collisions link1="axis_cam_top" link2="$(arg robot_name)_link_6" reason="Never" />
     <disable_collisions link1="axis_cam_top" link2="$(arg robot_name)_link_7" reason="Never" />
+    <disable_collisions link1="axis_cam_top" link2="$(arg robot_name)_link_ee" reason="Never" />
     <disable_collisions link1="axis_cam_top" link2="$(arg robot_name)_roboception_adapter" reason="Never" />
     <disable_collisions link1="axis_cam_top" link2="$(arg robot_name)_roboception_camera_uncal" reason="Never" />
@@ -99,5 +101,5 @@
     <disable_collisions link1="axis_cam_top" link2="wall_front" reason="Default" />
     <disable_collisions link1="axis_cam_top" link2="wall_left" reason="Never" />
-    <disable_collisions link1="axis_cam_top" link2="wall_right" reason="Never" />
+    <disable_collisions link1="axis_cam_top" link2="wall_right" reason="Default" />
     <disable_collisions link1="$(arg robot_name)_base_adapter" link2="$(arg robot_name)_link_0" reason="Adjacent" />
     <disable_collisions link1="$(arg robot_name)_base_adapter" link2="$(arg robot_name)_link_1" reason="Never" />
@@ -119,5 +121,4 @@
     <disable_collisions link1="$(arg robot_name)_gripper_adapter" link2="$(arg robot_name)_gripper_waggon_left" reason="Never" />
     <disable_collisions link1="$(arg robot_name)_gripper_adapter" link2="$(arg robot_name)_gripper_waggon_right" reason="Never" />
-    <disable_collisions link1="$(arg robot_name)_gripper_adapter" link2="$(arg robot_name)_link_0" reason="Never" />
     <disable_collisions link1="$(arg robot_name)_gripper_adapter" link2="$(arg robot_name)_link_1" reason="Never" />
     <disable_collisions link1="$(arg robot_name)_gripper_adapter" link2="$(arg robot_name)_link_2" reason="Never" />
@@ -126,5 +127,6 @@
     <disable_collisions link1="$(arg robot_name)_gripper_adapter" link2="$(arg robot_name)_link_5" reason="Never" />
     <disable_collisions link1="$(arg robot_name)_gripper_adapter" link2="$(arg robot_name)_link_6" reason="Never" />
-    <disable_collisions link1="$(arg robot_name)_gripper_adapter" link2="$(arg robot_name)_link_7" reason="Adjacent" />
+    <disable_collisions link1="$(arg robot_name)_gripper_adapter" link2="$(arg robot_name)_link_7" reason="Never" />
+    <disable_collisions link1="$(arg robot_name)_gripper_adapter" link2="$(arg robot_name)_link_ee" reason="Adjacent" />
     <disable_collisions link1="$(arg robot_name)_gripper_adapter" link2="$(arg robot_name)_roboception_adapter" reason="Never" />
     <disable_collisions link1="$(arg robot_name)_gripper_adapter" link2="$(arg robot_name)_roboception_camera_uncal" reason="Never" />
@@ -135,11 +137,10 @@
     <disable_collisions link1="$(arg robot_name)_gripper_base" link2="$(arg robot_name)_gripper_waggon_left" reason="Adjacent" />
     <disable_collisions link1="$(arg robot_name)_gripper_base" link2="$(arg robot_name)_gripper_waggon_right" reason="Adjacent" />
-    <disable_collisions link1="$(arg robot_name)_gripper_base" link2="$(arg robot_name)_link_1" reason="Never" />
     <disable_collisions link1="$(arg robot_name)_gripper_base" link2="$(arg robot_name)_link_2" reason="Never" />
-    <disable_collisions link1="$(arg robot_name)_gripper_base" link2="$(arg robot_name)_link_3" reason="Never" />
     <disable_collisions link1="$(arg robot_name)_gripper_base" link2="$(arg robot_name)_link_4" reason="Never" />
     <disable_collisions link1="$(arg robot_name)_gripper_base" link2="$(arg robot_name)_link_5" reason="Never" />
     <disable_collisions link1="$(arg robot_name)_gripper_base" link2="$(arg robot_name)_link_6" reason="Never" />
     <disable_collisions link1="$(arg robot_name)_gripper_base" link2="$(arg robot_name)_link_7" reason="Never" />
+    <disable_collisions link1="$(arg robot_name)_gripper_base" link2="$(arg robot_name)_link_ee" reason="Never" />
     <disable_collisions link1="$(arg robot_name)_gripper_base" link2="$(arg robot_name)_roboception_adapter" reason="Never" />
     <disable_collisions link1="$(arg robot_name)_gripper_base" link2="$(arg robot_name)_roboception_gusset" reason="Never" />
@@ -148,17 +149,18 @@
     <disable_collisions link1="$(arg robot_name)_gripper_finger_left" link2="$(arg robot_name)_gripper_waggon_left" reason="Adjacent" />
     <disable_collisions link1="$(arg robot_name)_gripper_finger_left" link2="$(arg robot_name)_gripper_waggon_right" reason="Never" />
-    <disable_collisions link1="$(arg robot_name)_gripper_finger_left" link2="$(arg robot_name)_link_3" reason="Never" />
     <disable_collisions link1="$(arg robot_name)_gripper_finger_left" link2="$(arg robot_name)_link_4" reason="Never" />
     <disable_collisions link1="$(arg robot_name)_gripper_finger_left" link2="$(arg robot_name)_link_5" reason="Never" />
     <disable_collisions link1="$(arg robot_name)_gripper_finger_left" link2="$(arg robot_name)_link_6" reason="Never" />
     <disable_collisions link1="$(arg robot_name)_gripper_finger_left" link2="$(arg robot_name)_link_7" reason="Never" />
+    <disable_collisions link1="$(arg robot_name)_gripper_finger_left" link2="$(arg robot_name)_link_ee" reason="Never" />
     <disable_collisions link1="$(arg robot_name)_gripper_finger_left" link2="$(arg robot_name)_roboception_adapter" reason="Never" />
     <disable_collisions link1="$(arg robot_name)_gripper_finger_right" link2="$(arg robot_name)_gripper_waggon_left" reason="Never" />
     <disable_collisions link1="$(arg robot_name)_gripper_finger_right" link2="$(arg robot_name)_gripper_waggon_right" reason="Adjacent" />
-    <disable_collisions link1="$(arg robot_name)_gripper_finger_right" link2="$(arg robot_name)_link_3" reason="Never" />
     <disable_collisions link1="$(arg robot_name)_gripper_finger_right" link2="$(arg robot_name)_link_4" reason="Never" />
     <disable_collisions link1="$(arg robot_name)_gripper_finger_right" link2="$(arg robot_name)_link_5" reason="Never" />
     <disable_collisions link1="$(arg robot_name)_gripper_finger_right" link2="$(arg robot_name)_link_6" reason="Never" />
     <disable_collisions link1="$(arg robot_name)_gripper_finger_right" link2="$(arg robot_name)_link_7" reason="Never" />
+    <disable_collisions link1="$(arg robot_name)_gripper_finger_right" link2="$(arg robot_name)_link_ee" reason="Never" />
+    <disable_collisions link1="$(arg robot_name)_gripper_finger_right" link2="$(arg robot_name)_roboception_adapter" reason="Never" />
     <disable_collisions link1="$(arg robot_name)_gripper_waggon_left" link2="$(arg robot_name)_gripper_waggon_right" reason="Never" />
     <disable_collisions link1="$(arg robot_name)_gripper_waggon_left" link2="$(arg robot_name)_link_1" reason="Never" />
@@ -169,8 +171,9 @@
     <disable_collisions link1="$(arg robot_name)_gripper_waggon_left" link2="$(arg robot_name)_link_6" reason="Never" />
     <disable_collisions link1="$(arg robot_name)_gripper_waggon_left" link2="$(arg robot_name)_link_7" reason="Never" />
+    <disable_collisions link1="$(arg robot_name)_gripper_waggon_left" link2="$(arg robot_name)_link_ee" reason="Never" />
     <disable_collisions link1="$(arg robot_name)_gripper_waggon_left" link2="$(arg robot_name)_roboception_adapter" reason="Never" />
+    <disable_collisions link1="$(arg robot_name)_gripper_waggon_left" link2="$(arg robot_name)_roboception_camera_uncal" reason="Never" />
     <disable_collisions link1="$(arg robot_name)_gripper_waggon_left" link2="$(arg robot_name)_roboception_gusset" reason="Never" />
     <disable_collisions link1="$(arg robot_name)_gripper_waggon_left" link2="profile_cams" reason="Never" />
-    <disable_collisions link1="$(arg robot_name)_gripper_waggon_right" link2="$(arg robot_name)_link_1" reason="Never" />
     <disable_collisions link1="$(arg robot_name)_gripper_waggon_right" link2="$(arg robot_name)_link_2" reason="Never" />
     <disable_collisions link1="$(arg robot_name)_gripper_waggon_right" link2="$(arg robot_name)_link_3" reason="Never" />
@@ -179,4 +182,5 @@
     <disable_collisions link1="$(arg robot_name)_gripper_waggon_right" link2="$(arg robot_name)_link_6" reason="Never" />
     <disable_collisions link1="$(arg robot_name)_gripper_waggon_right" link2="$(arg robot_name)_link_7" reason="Never" />
+    <disable_collisions link1="$(arg robot_name)_gripper_waggon_right" link2="$(arg robot_name)_link_ee" reason="Never" />
     <disable_collisions link1="$(arg robot_name)_gripper_waggon_right" link2="$(arg robot_name)_roboception_adapter" reason="Never" />
     <disable_collisions link1="$(arg robot_name)_gripper_waggon_right" link2="$(arg robot_name)_roboception_gusset" reason="Never" />
@@ -186,5 +190,4 @@
     <disable_collisions link1="$(arg robot_name)_link_0" link2="$(arg robot_name)_link_3" reason="Never" />
     <disable_collisions link1="$(arg robot_name)_link_0" link2="$(arg robot_name)_link_4" reason="Never" />
-    <disable_collisions link1="$(arg robot_name)_link_0" link2="$(arg robot_name)_link_7" reason="Never" />
     <disable_collisions link1="$(arg robot_name)_link_0" link2="$(arg robot_name)_roboception_adapter" reason="Never" />
     <disable_collisions link1="$(arg robot_name)_link_0" link2="$(arg robot_name)_roboception_camera_uncal" reason="Never" />
@@ -202,4 +205,5 @@
     <disable_collisions link1="$(arg robot_name)_link_1" link2="$(arg robot_name)_link_6" reason="Never" />
     <disable_collisions link1="$(arg robot_name)_link_1" link2="$(arg robot_name)_link_7" reason="Never" />
+    <disable_collisions link1="$(arg robot_name)_link_1" link2="$(arg robot_name)_link_ee" reason="Never" />
     <disable_collisions link1="$(arg robot_name)_link_1" link2="$(arg robot_name)_roboception_adapter" reason="Never" />
     <disable_collisions link1="$(arg robot_name)_link_1" link2="$(arg robot_name)_roboception_camera_uncal" reason="Never" />
@@ -216,4 +220,5 @@
     <disable_collisions link1="$(arg robot_name)_link_2" link2="$(arg robot_name)_link_6" reason="Never" />
     <disable_collisions link1="$(arg robot_name)_link_2" link2="$(arg robot_name)_link_7" reason="Never" />
+    <disable_collisions link1="$(arg robot_name)_link_2" link2="$(arg robot_name)_link_ee" reason="Never" />
     <disable_collisions link1="$(arg robot_name)_link_2" link2="$(arg robot_name)_roboception_adapter" reason="Never" />
     <disable_collisions link1="$(arg robot_name)_link_2" link2="$(arg robot_name)_roboception_camera_uncal" reason="Never" />
@@ -226,7 +231,8 @@
     <disable_collisions link1="$(arg robot_name)_link_2" link2="wall_right" reason="Never" />
     <disable_collisions link1="$(arg robot_name)_link_3" link2="$(arg robot_name)_link_4" reason="Adjacent" />
-    <disable_collisions link1="$(arg robot_name)_link_3" link2="$(arg robot_name)_link_5" reason="Never" />
+    <disable_collisions link1="$(arg robot_name)_link_3" link2="$(arg robot_name)_link_5" reason="Adjacent" />
     <disable_collisions link1="$(arg robot_name)_link_3" link2="$(arg robot_name)_link_6" reason="Never" />
     <disable_collisions link1="$(arg robot_name)_link_3" link2="$(arg robot_name)_link_7" reason="Never" />
+    <disable_collisions link1="$(arg robot_name)_link_3" link2="$(arg robot_name)_link_ee" reason="Never" />
     <disable_collisions link1="$(arg robot_name)_link_3" link2="$(arg robot_name)_roboception_adapter" reason="Never" />
     <disable_collisions link1="$(arg robot_name)_link_3" link2="$(arg robot_name)_roboception_camera_uncal" reason="Never" />
@@ -240,26 +246,36 @@
     <disable_collisions link1="$(arg robot_name)_link_4" link2="$(arg robot_name)_link_6" reason="Never" />
     <disable_collisions link1="$(arg robot_name)_link_4" link2="$(arg robot_name)_link_7" reason="Never" />
+    <disable_collisions link1="$(arg robot_name)_link_4" link2="$(arg robot_name)_link_ee" reason="Never" />
     <disable_collisions link1="$(arg robot_name)_link_4" link2="$(arg robot_name)_roboception_adapter" reason="Never" />
     <disable_collisions link1="$(arg robot_name)_link_4" link2="$(arg robot_name)_roboception_camera_uncal" reason="Never" />
     <disable_collisions link1="$(arg robot_name)_link_4" link2="$(arg robot_name)_roboception_gusset" reason="Never" />
     <disable_collisions link1="$(arg robot_name)_link_4" link2="profile_cams" reason="Never" />
+    <disable_collisions link1="$(arg robot_name)_link_4" link2="table" reason="Never" />
     <disable_collisions link1="$(arg robot_name)_link_4" link2="wall_front" reason="Never" />
     <disable_collisions link1="$(arg robot_name)_link_4" link2="wall_left" reason="Never" />
     <disable_collisions link1="$(arg robot_name)_link_4" link2="wall_right" reason="Never" />
     <disable_collisions link1="$(arg robot_name)_link_5" link2="$(arg robot_name)_link_6" reason="Adjacent" />
-    <disable_collisions link1="$(arg robot_name)_link_5" link2="$(arg robot_name)_link_7" reason="Adjacent" />
+    <disable_collisions link1="$(arg robot_name)_link_5" link2="$(arg robot_name)_link_7" reason="Default" />
+    <disable_collisions link1="$(arg robot_name)_link_5" link2="$(arg robot_name)_link_ee" reason="Default" />
     <disable_collisions link1="$(arg robot_name)_link_5" link2="$(arg robot_name)_roboception_adapter" reason="Never" />
     <disable_collisions link1="$(arg robot_name)_link_5" link2="$(arg robot_name)_roboception_camera_uncal" reason="Never" />
     <disable_collisions link1="$(arg robot_name)_link_5" link2="$(arg robot_name)_roboception_gusset" reason="Never" />
     <disable_collisions link1="$(arg robot_name)_link_5" link2="profile_cams" reason="Never" />
+    <disable_collisions link1="$(arg robot_name)_link_5" link2="wall_front" reason="Never" />
     <disable_collisions link1="$(arg robot_name)_link_6" link2="$(arg robot_name)_link_7" reason="Adjacent" />
+    <disable_collisions link1="$(arg robot_name)_link_6" link2="$(arg robot_name)_link_ee" reason="Default" />
     <disable_collisions link1="$(arg robot_name)_link_6" link2="$(arg robot_name)_roboception_adapter" reason="Never" />
     <disable_collisions link1="$(arg robot_name)_link_6" link2="$(arg robot_name)_roboception_camera_uncal" reason="Never" />
     <disable_collisions link1="$(arg robot_name)_link_6" link2="$(arg robot_name)_roboception_gusset" reason="Never" />
     <disable_collisions link1="$(arg robot_name)_link_6" link2="profile_cams" reason="Never" />
+    <disable_collisions link1="$(arg robot_name)_link_7" link2="$(arg robot_name)_link_ee" reason="Adjacent" />
     <disable_collisions link1="$(arg robot_name)_link_7" link2="$(arg robot_name)_roboception_adapter" reason="Never" />
     <disable_collisions link1="$(arg robot_name)_link_7" link2="$(arg robot_name)_roboception_camera_uncal" reason="Never" />
     <disable_collisions link1="$(arg robot_name)_link_7" link2="$(arg robot_name)_roboception_gusset" reason="Never" />
     <disable_collisions link1="$(arg robot_name)_link_7" link2="profile_cams" reason="Never" />
+    <disable_collisions link1="$(arg robot_name)_link_ee" link2="$(arg robot_name)_roboception_adapter" reason="Never" />
+    <disable_collisions link1="$(arg robot_name)_link_ee" link2="$(arg robot_name)_roboception_camera_uncal" reason="Never" />
+    <disable_collisions link1="$(arg robot_name)_link_ee" link2="$(arg robot_name)_roboception_gusset" reason="Never" />
+    <disable_collisions link1="$(arg robot_name)_link_ee" link2="profile_cams" reason="Never" />
     <disable_collisions link1="$(arg robot_name)_roboception_adapter" link2="$(arg robot_name)_roboception_camera_uncal" reason="Adjacent" />
     <disable_collisions link1="$(arg robot_name)_roboception_adapter" link2="$(arg robot_name)_roboception_gusset" reason="Adjacent" />
@@ -269,5 +285,5 @@
     <disable_collisions link1="$(arg robot_name)_roboception_adapter" link2="wall_front" reason="Default" />
     <disable_collisions link1="$(arg robot_name)_roboception_adapter" link2="wall_left" reason="Never" />
-    <disable_collisions link1="$(arg robot_name)_roboception_adapter" link2="wall_right" reason="Never" />
+    <disable_collisions link1="$(arg robot_name)_roboception_adapter" link2="wall_right" reason="Default" />
     <disable_collisions link1="$(arg robot_name)_roboception_camera_uncal" link2="$(arg robot_name)_roboception_gusset" reason="Default" />
     <disable_collisions link1="$(arg robot_name)_roboception_camera_uncal" link2="profile_cams" reason="Default" />
@@ -282,5 +298,5 @@
     <disable_collisions link1="$(arg robot_name)_roboception_gusset" link2="wall_front" reason="Default" />
     <disable_collisions link1="$(arg robot_name)_roboception_gusset" link2="wall_left" reason="Never" />
-    <disable_collisions link1="$(arg robot_name)_roboception_gusset" link2="wall_right" reason="Never" />
+    <disable_collisions link1="$(arg robot_name)_roboception_gusset" link2="wall_right" reason="Default" />
     <disable_collisions link1="profile_cams" link2="table" reason="Adjacent" />
     <disable_collisions link1="profile_cams" link2="wall_back" reason="Adjacent" />
