Commit message: add iiwa 7, egl 90 and rc_visard 160 description
Signed-off-by: Wolfgang Wiedmeyer <wolfgang.wiedmeyer@kit.edu>

File: rll_description/urdf/rll_setup.urdf.xacro (robot description, xacro)
@@ -1,9 +1,8 @@
 <?xml version="1.0"?>
 <robot xmlns:xacro="http://www.ros.org/wiki/xacro" name="iiwa7">
-  <!-- Import Rviz colors -->
-  <xacro:include filename="$(find iiwa_description)/urdf/materials.xacro" />
-  <xacro:include filename="$(find iiwa_description)/urdf/iiwa7.xacro"/>
-  <xacro:include filename="$(find schunk_gripper_egl90)/urdf/egl90_macro.xacro"/>
-  <xacro:include filename="$(find rc_visard_description)/urdf/rc_visard_160.xacro"/>
+  <xacro:include filename="$(find rll_description)/urdf/iiwa7/iiwa7.xacro"/>
+  <xacro:include filename="$(find rll_description)/urdf/iiwa7/materials.xacro" />
+  <xacro:include filename="$(find rll_description)/urdf/egl90/egl90_macro.xacro"/>
+  <xacro:include filename="$(find rll_description)/urdf/visard160/rc_visard_160.xacro"/>
   <!--  Arguments for the iiwa7 macro  -->
   <xacro:arg name="hardware_interface" default="PositionJointInterface"/>
@@ -172,5 +171,5 @@
       <origin xyz="0 0 0.024" rpy="${180 * PI / 180} 0 ${-90 * PI / 180}"/>
       <geometry>
-        <mesh filename="package://rll_description/meshes/visual/gripper_adapter.dae" scale="0.001 0.001 0.001"/>
+        <mesh filename="package://rll_description/meshes/egl90/visual/gripper_adapter.dae" scale="0.001 0.001 0.001"/>
       </geometry>
       <material name="Grey"/>
@@ -179,5 +178,5 @@
       <origin xyz="0 0 0.024" rpy="${180 * PI / 180} 0 ${-90 * PI / 180}"/>
       <geometry>
-        <mesh filename="package://rll_description/meshes/visual/gripper_adapter.dae" scale="0.001 0.001 0.001"/>
+        <mesh filename="package://rll_description/meshes/egl90/visual/gripper_adapter.dae" scale="0.001 0.001 0.001"/>
       </geometry>
       <material name="Grey"/>
@@ -188,5 +187,5 @@
   </xacro:egl90>
   <xacro:egl90-jaws prefix="$(arg robot_name)_" x="0.0" min="-0.015" max="0.026">
-    <mesh filename="package://rll_description/meshes/visual/gripper_finger.dae" scale="0.001 0.001 0.001"/>
+    <mesh filename="package://rll_description/meshes/egl90/visual/gripper_finger.dae" scale="0.001 0.001 0.001"/>
   </xacro:egl90-jaws>
   <!-- TCP link -->

Commit message: description: materials cleanup
Signed-off-by: Wolfgang Wiedmeyer <wolfgang.wiedmeyer@kit.edu>

File: rll_description/urdf/rll_setup.urdf.xacro (robot description, xacro)
@@ -2,5 +2,4 @@
 <robot xmlns:xacro="http://www.ros.org/wiki/xacro" name="iiwa7">
   <xacro:include filename="$(find rll_description)/urdf/iiwa7/iiwa7.xacro"/>
-  <xacro:include filename="$(find rll_description)/urdf/iiwa7/materials.xacro" />
   <xacro:include filename="$(find rll_description)/urdf/egl90/egl90_macro.xacro"/>
   <xacro:include filename="$(find rll_description)/urdf/visard160/rc_visard_160.xacro"/>
@@ -8,10 +7,4 @@
   <xacro:arg name="hardware_interface" default="PositionJointInterface"/>
   <xacro:arg name="robot_name" default="iiwa"/>
-  <material name="steel">
-    <color rgba="0.8784 0.8745 0.8588 1.0"/>
-  </material>
-  <material name="transparent">
-    <color rgba="0.8784 0.8745 0.8588 0.3"/>
-  </material>
   <!--  Define the origin of your 3D space
        Here we define a box lying at 0,0,0 with some dimensions. In reality, our robot is placed on top of a table.
@@ -34,5 +27,4 @@
         <box size="1.2 1.6 0.203"/>
       </geometry>
-      <material name="steel" />
     </collision>
   </link>
@@ -71,5 +63,4 @@
         <box size="0.01 1.6 1.1" rpy="0 0 0"/>
       </geometry>
-      <material name="transparent" />
     </collision>
   </link>
@@ -87,5 +78,4 @@
         <box size="0.01 1.6 1.1" rpy="0 0 0"/>
       </geometry>
-      <material name="transparent" />
     </collision>
   </link>
@@ -103,5 +93,4 @@
         <box size="1.2 0.01 1.1" rpy="0 0 0"/>
       </geometry>
-      <material name="transparent" />
     </collision>
   </link>
@@ -119,5 +108,4 @@
         <box size="1.2 0.01 1.1" rpy="0 0 0"/>
       </geometry>
-      <material name="transparent" />
     </collision>
   </link>
@@ -173,5 +161,4 @@
         <mesh filename="package://rll_description/meshes/egl90/visual/gripper_adapter.dae" scale="0.001 0.001 0.001"/>
       </geometry>
-      <material name="Grey"/>
     </visual>
     <collision>
@@ -180,5 +167,4 @@
         <mesh filename="package://rll_description/meshes/egl90/visual/gripper_adapter.dae" scale="0.001 0.001 0.001"/>
       </geometry>
-      <material name="Grey"/>
     </collision>
   </link>
@@ -252,6 +238,11 @@
         <box size="0.30 0.13 0.10" rpy="0 0 0"/>
       </geometry>
-      <material name="transparent" />
-    </collision>
-  </link>
+    </collision>
+  </link>
+  <material name="steel">
+    <color rgba="0.8784 0.8745 0.8588 1.0"/>
+  </material>
+  <material name="transparent">
+    <color rgba="0.8784 0.8745 0.8588 0.3"/>
+  </material>
 </robot>

Commit message: description: fix gripper adapter color in Gazebo
Signed-off-by: Wolfgang Wiedmeyer <wolfgang.wiedmeyer@kit.edu>

File: rll_description/urdf/rll_setup.urdf.xacro (robot description, xacro)
@@ -229,4 +229,8 @@
     <static>true</static>
   </gazebo>
+  <gazebo reference="$(arg robot_name)_gripper_adapter">
+    <material>Gazebo/Grey</material>
+    <static>true</static>
+  </gazebo>
   <material name="steel">
     <color rgba="0.8784 0.8745 0.8588 1.0"/>

Commit message: description: visual for table and base adapter
Thanks to Michael Mende for the models!

Signed-off-by: Wolfgang Wiedmeyer <wolfgang.wiedmeyer@kit.edu>

File: rll_description/urdf/rll_setup.urdf.xacro (robot description, xacro)
@@ -13,9 +13,8 @@
   <link name="world">
     <visual>
-      <origin xyz="0 0 -0.1" rpy="0 0 0"/>
-      <geometry>
-        <box size="1.2 1.6 0.2"/>
-      </geometry>
-      <material name="steel" />
+      <origin xyz="0 0 0" rpy="0 0 ${90 * PI / 180}"/>
+      <geometry>
+        <mesh filename="package://rll_description/meshes/rll/visual/table.dae"/>
+      </geometry>
     </visual>
     <collision>
@@ -117,9 +116,8 @@
   <link name="$(arg robot_name)_base_adapter">
     <visual>
-      <origin xyz="0 0 0.01" rpy="0 0 0"/>
-      <geometry>
-        <cylinder length="0.02" radius="0.16"/>
-      </geometry>
-      <material name="steel" />
+      <origin xyz="0 0 0" rpy="0 0 0"/>
+      <geometry>
+          <mesh filename="package://rll_description/meshes/rll/visual/base_adapter.dae"/>
+      </geometry>
     </visual>
     <collision>
@@ -225,10 +223,11 @@
     </collision>
   </link>
+  <gazebo reference="world">
+    <static>true</static>
+  </gazebo>
   <gazebo reference="$(arg robot_name)_base_adapter">
-    <material>Gazebo/Grey</material>
     <static>true</static>
   </gazebo>
   <gazebo reference="$(arg robot_name)_gripper_adapter">
-    <material>Gazebo/Grey</material>
     <static>true</static>
   </gazebo>

Commit message: description: new Roboception mount model and improved collision objects
Thanks again to Michael Mende for the Models!

Signed-off-by: Wolfgang Wiedmeyer <wolfgang.wiedmeyer@kit.edu>

File: rll_description/urdf/rll_setup.urdf.xacro (robot description, xacro)
@@ -60,5 +60,5 @@
       <origin xyz="0 0 0" rpy="0 0 0"/>
       <geometry>
-        <box size="0.01 1.6 1.1" rpy="0 0 0"/>
+        <box size="0.01 1.6 1.4" rpy="0 0 0"/>
       </geometry>
     </collision>
@@ -75,5 +75,5 @@
       <origin xyz="0 0 0" rpy="0 0 0"/>
       <geometry>
-        <box size="0.01 1.6 1.1" rpy="0 0 0"/>
+        <box size="0.01 1.6 1.4" rpy="0 0 0"/>
       </geometry>
     </collision>
@@ -90,5 +90,5 @@
       <origin xyz="0 0 0" rpy="0 0 0"/>
       <geometry>
-        <box size="1.2 0.01 1.1" rpy="0 0 0"/>
+        <box size="1.2 0.01 1.4" rpy="0 0 0"/>
       </geometry>
     </collision>
@@ -105,5 +105,5 @@
       <origin xyz="0 0 0" rpy="0 0 0"/>
       <geometry>
-        <box size="1.2 0.01 1.1" rpy="0 0 0"/>
+        <box size="1.2 0.01 1.4" rpy="0 0 0"/>
       </geometry>
     </collision>
@@ -186,41 +186,59 @@
     </actuator>
   </transmission>
+  <joint name="profile_cams_joint" type="fixed">
+    <parent link="world" />
+    <child link="profile_cams" />
+    <origin xyz="0 0 0" rpy="0 0 0"/>
+  </joint>
+  <link name="profile_cams">
+    <visual>
+      <origin xyz="0 0 0" rpy="0 0 ${90 * PI / 180}"/>
+      <geometry>
+        <mesh filename="package://rll_description/meshes/rll/visual/profile_cams.dae"/>
+      </geometry>
+    </visual>
+    <collision>
+      <origin xyz="0.58 0.82 0.17" rpy="0 0 0"/>
+      <geometry>
+        <box size="0.05 0.05 2.0"/>
+      </geometry>
+    </collision>
+  </link>
+  <joint name="roboception_gusset_joint" type="fixed">
+    <parent link="profile_cams" />
+    <child link="roboception_gusset" />
+    <origin xyz="0.577 0.8 0.825" rpy="0 ${180 * PI / 180} 0"/>
+  </joint>
+  <link name="roboception_gusset">
+    <visual>
+      <origin xyz="0 0 0" rpy="0 0 0"/>
+      <geometry>
+        <mesh filename="package://rll_description/meshes/rll/visual/roboception_gusset.dae"/>
+      </geometry>
+    </visual>
+    <collision>
+      <origin xyz="0 -0.05 0.05" rpy="0 0 0"/>
+      <geometry>
+        <box size="0.05 0.1 0.1"/>
+      </geometry>
+    </collision>
+  </link>
   <!-- Roboception camera -->
-  <joint name="roboception_base_joint" type="fixed">
-    <parent link="world" />
-    <child link="roboception_base" />
-    <origin xyz="0.52 0.72 0.74" rpy="0 0 ${135 * PI / 180}"/>
-  </joint>
-  <link name="roboception_base">
-    <visual>
-      <origin xyz="0 0 0.04" rpy="0 0 0"/>
-      <geometry>
-        <cylinder length="0.08" radius="0.03"/>
-      </geometry>
-      <material name="steel" />
-    </visual>
-    <collision>
-      <origin xyz="0 0 0.04" rpy="0 0 0"/>
-      <geometry>
-        <cylinder length="0.08" radius="0.03"/>
-      </geometry>
-    </collision>
-  </link>
-  <xacro:rc_160 parent="roboception_base" prefix="$(arg robot_name)_">
-    <origin xyz="-0.08 0.03 0.1" rpy="${-135 * PI / 180} 0 0"/>
+  <joint name="roboception_adapter_joint" type="fixed">
+    <parent link="roboception_gusset" />
+    <child link="roboception_adapter" />
+    <origin xyz="0.03 -0.075 0" rpy="${-90 * PI / 180} 0 ${135 * PI / 180}"/>
+  </joint>
+  <link name="roboception_adapter">
+    <visual>
+      <origin xyz="0 0 0" rpy="0 0 0"/>
+      <geometry>
+        <mesh filename="package://rll_description/meshes/rll/visual/roboception_adapter.dae"/>
+      </geometry>
+    </visual>
+  </link>
+  <xacro:rc_160 parent="roboception_adapter" prefix="$(arg robot_name)_">
+    <origin xyz="-0.03 0.03 -0.08" rpy="${45 * PI / 180} ${-90 * PI / 180} 0"/>
   </xacro:rc_160>
-  <joint name="roboception_collision_joint" type="fixed">
-    <parent link="world" />
-    <child link="roboception_collision" />
-    <origin xyz="0.52 0.72 0.74" rpy="0 0 ${135 * PI / 180}"/>
-  </joint>
-  <link name="roboception_collision">
-    <collision>
-      <origin xyz="-0.0 0.03 0.1" rpy="${-135 * PI / 180} 0 0"/>
-      <geometry>
-        <box size="0.30 0.13 0.10" rpy="0 0 0"/>
-      </geometry>
-    </collision>
-  </link>
   <gazebo reference="world">
     <static>true</static>
@@ -232,7 +250,4 @@
     <static>true</static>
   </gazebo>
-  <material name="steel">
-    <color rgba="0.8784 0.8745 0.8588 1.0"/>
-  </material>
   <material name="transparent">
     <color rgba="0.8784 0.8745 0.8588 0.3"/>

File: rll_description/urdf/visard160/rc_visard_160.xacro (robot description, xacro)
@@ -14,6 +14,7 @@
       </visual>
       <collision>
+          <origin xyz="0.08 0.03 -0.05" rpy="0 0 0"/>
           <geometry>
-              <mesh filename="package://rll_description/meshes/visard160/collision/rc_visard_160.stl"/>
+              <box size="0.27 0.2 0.27"/>
           </geometry>
       </collision>
