Commit message: description: improve Roboception camera position
Signed-off-by: Wolfgang Wiedmeyer <wolfgang.wiedmeyer@kit.edu>

File: rll_description/urdf/rll_cell.xacro (robot description, xacro)
@@ -96,5 +96,5 @@
     <!-- Roboception camera -->
     <xacro:rc_160 parent="profile_cams" prefix="$(arg robot_name)_">
-      <origin xyz="0.577 0.8 0.825" rpy="0 ${180 * pi / 180} 0"/>
+      <origin xyz="0.577 0.8 0.829" rpy="0 ${180 * pi / 180} 0"/>
     </xacro:rc_160>
     <!-- Axis camera -->

File: rll_description/urdf/visard160/rc_visard_160.xacro (robot description, xacro)
@@ -24,5 +24,5 @@
       <parent link="${prefix}roboception_gusset" />
       <child link="${prefix}roboception_adapter" />
-      <origin xyz="0.03 -0.075 0" rpy="${-90 * pi / 180} 0 ${135 * pi / 180}"/>
+      <origin xyz="0.015 -0.075 0" rpy="${-90 * pi / 180} 0 ${125 * pi / 180}"/>
     </joint>
     <link name="${prefix}roboception_adapter">
@@ -37,5 +37,5 @@
       <parent link="${prefix}roboception_adapter"/>
       <child link="${prefix}roboception_camera"/>
-      <origin xyz="-0.03 0.03 -0.08" rpy="${45 * pi / 180} ${-90 * pi / 180} 0"/>
+      <origin xyz="-0.031 0.0375 0.08" rpy="${-45 * pi / 180} ${90 * pi / 180} ${180 * pi / 180}"/>
     </joint>
     <link name="${prefix}roboception_camera">
@@ -52,10 +52,4 @@
       </collision>
     </link>
-    <link name="${prefix}roboception_mounting"/>
-    <joint name="${prefix}mounting_to_camera" type="fixed">
-      <parent link="${prefix}roboception_camera"/>
-      <child link="${prefix}roboception_mounting"/>
-      <origin xyz="0.080 0.0375 -0.031" />
-    </joint>
   </xacro:macro>
 </robot>
