Commit message: description: remove visuals for virtual walls
They are confusing and annoying when using the interactive marker in RViz to move the robot.

Signed-off-by: Wolfgang Wiedmeyer <wolfgang.wiedmeyer@kit.edu>

File: rll_description/urdf/rll_virtual.xacro (robot description, xacro)
@@ -24,11 +24,4 @@
     </joint>
     <link name="wall_front">
-      <visual>
-        <origin xyz="0 0 0" rpy="0 0 0"/>
-        <geometry>
-          <box size="0.01 0.8 0.55" rpy="0 0 0"/>
-        </geometry>
-        <material name="transparent" />
-      </visual>
       <collision>
         <origin xyz="0 0 0" rpy="0 0 0"/>
@@ -39,11 +32,4 @@
     </link>
     <link name="wall_back">
-      <visual>
-        <origin xyz="0 0 0" rpy="0 0 0"/>
-        <geometry>
-          <box size="0.01 0.8 0.55" rpy="0 0 0"/>
-        </geometry>
-        <material name="transparent" />
-      </visual>
       <collision>
         <origin xyz="0 0 0" rpy="0 0 0"/>
@@ -54,11 +40,4 @@
     </link>
     <link name="wall_left">
-      <visual>
-        <origin xyz="0 0 0" rpy="0 0 0"/>
-        <geometry>
-          <box size="0.6 0.01 0.55" rpy="0 0 0"/>
-        </geometry>
-        <material name="transparent" />
-      </visual>
       <collision>
         <origin xyz="0 0 0" rpy="0 0 0"/>
@@ -69,11 +48,4 @@
     </link>
     <link name="wall_right">
-      <visual>
-        <origin xyz="0 0 0" rpy="0 0 0"/>
-        <geometry>
-          <box size="0.6 0.01 0.55" rpy="0 0 0"/>
-        </geometry>
-        <material name="transparent" />
-      </visual>
       <collision>
         <origin xyz="0 0 0" rpy="0 0 0"/>

Commit message: desc: move side and back walls 7cm to the inside
Signed-off-by: Wolfgang Wiedmeyer <wolfgang.wiedmeyer@kit.edu>

File: rll_description/urdf/rll_virtual.xacro (robot description, xacro)
@@ -3,4 +3,12 @@
   <xacro:macro name="rll_virtual">
     <!-- virtual walls -->
+    <!-- the front wall is exactly at the border of the table while the other -->
+    <!-- walls are moved 7cm away from the table border towards the world frame. -->
+    <!-- The Sunrise collision model uses spheres which is a lot less accurate -->
+    <!-- than the MoveIt collision model. To account for the differences, this -->
+    <!-- 7cm offset is introduced. -->
+    <!-- TODO: The front wall stays at the border because otherwise current Playground -->
+    <!--       project code would break. But the wall also needs to be moved inside when -->
+    <!--       something gets mounted to the front part of the table. -->
     <joint name="wall_joint1" type="fixed">
       <parent link="world" />
@@ -11,15 +19,15 @@
       <parent link="world" />
       <child link="wall_back" />
-      <origin xyz="-0.605 0 0.7" rpy="0 0 0"/>
+      <origin xyz="-0.535 0 0.7" rpy="0 0 0"/>
     </joint>
     <joint name="wall_joint3" type="fixed">
       <parent link="world" />
       <child link="wall_left" />
-      <origin xyz="0 -0.805 0.7" rpy="0 0 0"/>
+      <origin xyz="0 -0.735 0.7" rpy="0 0 0"/>
     </joint>
     <joint name="wall_joint4" type="fixed">
       <parent link="world" />
       <child link="wall_right" />
-      <origin xyz="0 0.805 0.7" rpy="0 0 0"/>
+      <origin xyz="0 0.735 0.7" rpy="0 0 0"/>
     </joint>
     <link name="wall_front">

Commit message: Revert "desc: move side and back walls 7cm to the inside"
This should not be necessary anymore with the addition of the simplified
iiwa collision model. The iiwa collision model is now compatible with the
Kuka Sunrise model.

This reverts commit 591111bc5bc6c9616290a0cdf16cf9a9302d750e.

Signed-off-by: Wolfgang Wiedmeyer <wolfgang.wiedmeyer@kit.edu>

File: rll_description/urdf/rll_virtual.xacro (robot description, xacro)
@@ -3,12 +3,4 @@
   <xacro:macro name="rll_virtual">
     <!-- virtual walls -->
-    <!-- the front wall is exactly at the border of the table while the other -->
-    <!-- walls are moved 7cm away from the table border towards the world frame. -->
-    <!-- The Sunrise collision model uses spheres which is a lot less accurate -->
-    <!-- than the MoveIt collision model. To account for the differences, this -->
-    <!-- 7cm offset is introduced. -->
-    <!-- TODO: The front wall stays at the border because otherwise current Playground -->
-    <!--       project code would break. But the wall also needs to be moved inside when -->
-    <!--       something gets mounted to the front part of the table. -->
     <joint name="wall_joint1" type="fixed">
       <parent link="world" />
@@ -19,15 +11,15 @@
       <parent link="world" />
       <child link="wall_back" />
-      <origin xyz="-0.535 0 0.7" rpy="0 0 0"/>
+      <origin xyz="-0.605 0 0.7" rpy="0 0 0"/>
     </joint>
     <joint name="wall_joint3" type="fixed">
       <parent link="world" />
       <child link="wall_left" />
-      <origin xyz="0 -0.735 0.7" rpy="0 0 0"/>
+      <origin xyz="0 -0.805 0.7" rpy="0 0 0"/>
     </joint>
     <joint name="wall_joint4" type="fixed">
       <parent link="world" />
       <child link="wall_right" />
-      <origin xyz="0 0.735 0.7" rpy="0 0 0"/>
+      <origin xyz="0 0.805 0.7" rpy="0 0 0"/>
     </joint>
     <link name="wall_front">
