Commit message: WIP: description: add Axis webcam and refactoring
Signed-off-by: Wolfgang Wiedmeyer <wolfgang.wiedmeyer@kit.edu>

File: rll_description/urdf/rll.gazebo.xacro (robot description, xacro)
@@ -2,21 +2,9 @@
 <robot xmlns:xacro="http://www.ros.org/wiki/xacro">
   <xacro:macro name="rll_gazebo" params="robot_name">
-  <gazebo reference="world">
-    <static>true</static>
-  </gazebo>
   <!-- Link Table -->
   <gazebo reference="table">
     <static>true</static>
   </gazebo>
-  <!-- Link iiwa_base_adapter -->
-  <gazebo reference="$(arg robot_name)_base_adapter">
-    <static>true</static>
-  </gazebo>
-  <!-- Link roboception_adapter -->
-  <gazebo reference="roboception_adapter">
-    <static>true</static>
-  </gazebo>
-  <!-- Link roboception_gusset -->
-  <gazebo reference="roboception_gusset">
+  <gazebo reference="$(arg robot_name)_link_0">
     <static>true</static>
   </gazebo>

File: rll_description/urdf/rll_main.urdf.xacro (robot description, xacro)
@@ -4,4 +4,5 @@
   <xacro:include filename="$(find rll_description)/urdf/egl90/egl90_macro.xacro"/>
   <xacro:include filename="$(find rll_description)/urdf/visard160/rc_visard_160.xacro"/>
+  <xacro:include filename="$(find rll_description)/urdf/rll_virtual.xacro"/>
   <xacro:include filename="$(find rll_description)/urdf/rll.gazebo.xacro"/>
   <xacro:include filename="$(find rll_description)/urdf/rll.transmission.xacro"/>
@@ -34,85 +35,4 @@
         <!-- for grasping objects on table -->
         <box size="1.2 1.6 0.203"/>
-      </geometry>
-    </collision>
-  </link>
-  <!-- virtual walls -->
-  <joint name="wall_joint1" type="fixed">
-    <parent link="world" />
-    <child link="wall_front" />
-    <origin xyz="0.605 0 0.7" rpy="0 0 0"/>
-  </joint>
-  <joint name="wall_joint2" type="fixed">
-    <parent link="world" />
-    <child link="wall_back" />
-    <origin xyz="-0.605 0 0.7" rpy="0 0 0"/>
-  </joint>
-  <joint name="wall_joint3" type="fixed">
-    <parent link="world" />
-    <child link="wall_left" />
-    <origin xyz="0 -0.805 0.7" rpy="0 0 0"/>
-  </joint>
-  <joint name="wall_joint4" type="fixed">
-    <parent link="world" />
-    <child link="wall_right" />
-    <origin xyz="0 0.805 0.7" rpy="0 0 0"/>
-  </joint>
-  <link name="wall_front">
-    <visual>
-      <origin xyz="0 0 0" rpy="0 0 0"/>
-      <geometry>
-        <box size="0.01 0.8 0.55" rpy="0 0 0"/>
-      </geometry>
-      <material name="transparent" />
-    </visual>
-    <collision>
-      <origin xyz="0 0 0" rpy="0 0 0"/>
-      <geometry>
-        <box size="0.01 1.6 1.4" rpy="0 0 0"/>
-      </geometry>
-    </collision>
-  </link>
-  <link name="wall_back">
-    <visual>
-      <origin xyz="0 0 0" rpy="0 0 0"/>
-      <geometry>
-        <box size="0.01 0.8 0.55" rpy="0 0 0"/>
-      </geometry>
-      <material name="transparent" />
-    </visual>
-    <collision>
-      <origin xyz="0 0 0" rpy="0 0 0"/>
-      <geometry>
-        <box size="0.01 1.6 1.4" rpy="0 0 0"/>
-      </geometry>
-    </collision>
-  </link>
-  <link name="wall_left">
-    <visual>
-      <origin xyz="0 0 0" rpy="0 0 0"/>
-      <geometry>
-        <box size="0.6 0.01 0.55" rpy="0 0 0"/>
-      </geometry>
-      <material name="transparent" />
-    </visual>
-    <collision>
-      <origin xyz="0 0 0" rpy="0 0 0"/>
-      <geometry>
-        <box size="1.2 0.01 1.4" rpy="0 0 0"/>
-      </geometry>
-    </collision>
-  </link>
-  <link name="wall_right">
-    <visual>
-      <origin xyz="0 0 0" rpy="0 0 0"/>
-      <geometry>
-        <box size="0.6 0.01 0.55" rpy="0 0 0"/>
-      </geometry>
-      <material name="transparent" />
-    </visual>
-    <collision>
-      <origin xyz="0 0 0" rpy="0 0 0"/>
-      <geometry>
-        <box size="1.2 0.01 1.4" rpy="0 0 0"/>
       </geometry>
     </collision>
@@ -161,4 +81,9 @@
   </joint>
   <link name="profile_cams">
+    <inertial>
+       <origin xyz="0 0 0" rpy="0 0 0"/>
+       <mass value="0.1"/>
+       <inertia ixx="0.0001" ixy="0" ixz="0" iyy="0.0002" iyz="0" izz="0.0001"/>
+    </inertial>
     <visual>
       <origin xyz="0 0 0" rpy="0 0 ${90 * pi / 180}"/>
@@ -178,8 +103,45 @@
     <origin xyz="0.577 0.8 0.825" rpy="0 ${180 * pi / 180} 0"/>
   </xacro:rc_160>
-  <material name="transparent">
-    <color rgba="0.8784 0.8745 0.8588 0.3"/>
-  </material>
+  <!-- Axis camera -->
+  <joint name="axis_cam_base_joint" type="fixed">
+    <parent link="profile_cams" />
+    <child link="axis_cam_base" />
+    <origin xyz="0.577 0.8 1.13" rpy="${90 * pi / 180} 0 0"/>
+  </joint>
+  <link name="axis_cam_base">
+    <visual>
+      <origin xyz="0 0 0" rpy="0 0 0"/>
+      <geometry>
+        <mesh filename="package://rll_description/meshes/rll/visual/axis_cam_bottom.dae"/>
+      </geometry>
+    </visual>
+    <collision>
+      <origin xyz="0 0 0.035" rpy="0 0 0"/>
+      <geometry>
+        <box size="0.01 0.01 0.07"/>
+      </geometry>
+    </collision>
+  </link>
+  <joint name="axis_cam_top_joint" type="fixed">
+    <parent link="axis_cam_base" />
+    <child link="axis_cam_top" />
+    <origin xyz="0 0 0.068" rpy="${30 * pi / 180} ${30 * pi / 180} ${-65 * pi / 180}"/>
+  </joint>
+  <link name="axis_cam_top">
+    <visual>
+      <origin xyz="0 0 0" rpy="0 0 0"/>
+      <geometry>
+        <mesh filename="package://rll_description/meshes/rll/visual/axis_cam_top.dae"/>
+      </geometry>
+    </visual>
+    <collision>
+      <origin xyz="0 0.01 0.03" rpy="0 0 0"/>
+      <geometry>
+        <box size="0.06 0.11 0.06"/>
+      </geometry>
+    </collision>
+  </link>
   <!--Extensions -->
+  <xacro:rll_virtual />
   <xacro:rll_gazebo robot_name="$(arg robot_name)" />
   <xacro:rll_transmission hardware_interface="$(arg hardware_interface)" robot_name="$(arg robot_name)"/>

Commit message: allow to load an extended description based on rll_cell
Signed-off-by: Wolfgang Wiedmeyer <wolfgang.wiedmeyer@kit.edu>

File: rll_description/urdf/rll.gazebo.xacro (robot description, xacro)
@@ -4,4 +4,6 @@
   <!-- Link Table -->
   <gazebo reference="table">
+    <mu1>1.0</mu1>
+    <mu2>1.0</mu2>
     <static>true</static>
   </gazebo>

File: rll_description/urdf/rll_main.urdf.xacro (robot description, xacro)
@@ -1,143 +1,7 @@
 <?xml version="1.0"?>
 <robot xmlns:xacro="http://www.ros.org/wiki/xacro" name="rll_cell">
-  <xacro:include filename="$(find rll_description)/urdf/iiwa7/iiwa7.xacro"/>
-  <xacro:include filename="$(find rll_description)/urdf/egl90/egl90_macro.xacro"/>
-  <xacro:include filename="$(find rll_description)/urdf/visard160/rc_visard_160.xacro"/>
-  <xacro:include filename="$(find rll_description)/urdf/rll_virtual.xacro"/>
-  <xacro:include filename="$(find rll_description)/urdf/rll.gazebo.xacro"/>
-  <xacro:include filename="$(find rll_description)/urdf/rll.transmission.xacro"/>
-  <!--  Arguments for the iiwa7 macro  -->
+  <xacro:include filename="$(find rll_description)/urdf/rll_cell.xacro"/>
   <xacro:arg name="hardware_interface" default="PositionJointInterface"/>
   <xacro:arg name="robot_name" default="iiwa"/>
-  <link name="world"/>
-  <joint name="table_joint" type="fixed">
-    <parent link="world" />
-    <child link="table" />
-    <origin xyz="0 0 0" rpy="0 0 0"/>
-  </joint>
-  <link name="table">
-    <inertial>
-      <origin xyz="0 0 0" rpy="0 0 0"/>
-      <mass value="0.1"/>
-      <inertia ixx="0.0001" ixy="0" ixz="0" iyy="0.0002" iyz="0" izz="0.0001"/>
-    </inertial>
-    <visual>
-      <origin xyz="0 0 0" rpy="0 0 ${90 * pi / 180}"/>
-      <geometry>
-        <mesh filename="package://rll_description/meshes/rll/visual/table.dae"/>
-      </geometry>
-    </visual>
-    <collision>
-      <origin xyz="0 0 -0.1" rpy="0 0 0"/>
-      <geometry>
-        <!-- for disallowing eef positions below joint 1 -->
-        <!-- <box size="1.2 1.6 0.49"/> -->
-        <!-- for grasping objects on table -->
-        <box size="1.2 1.6 0.203"/>
-      </geometry>
-    </collision>
-  </link>
-  <joint name="base_adapter_joint" type="fixed">
-    <parent link="world" />
-    <child link="$(arg robot_name)_base_adapter" />
-    <origin xyz="-0.2 0 0" rpy="0 0 0"/>
-  </joint>
-  <link name="$(arg robot_name)_base_adapter">
-    <visual>
-      <origin xyz="0 0 0" rpy="0 0 0"/>
-      <geometry>
-        <mesh filename="package://rll_description/meshes/rll/visual/base_adapter.dae"/>
-      </geometry>
-    </visual>
-    <collision>
-      <origin xyz="0 0 0.01" rpy="0 0 0"/>
-      <geometry>
-        <cylinder length="0.02" radius="0.16"/>
-      </geometry>
-    </collision>
-  </link>
-  <!-- Here we insert an iiwa7 robot in the scene, it's origin is on top of the adapter. -->
-  <xacro:iiwa7 hardware_interface="$(arg hardware_interface)" robot_name="$(arg robot_name)" parent="$(arg robot_name)_base_adapter">
-    <origin xyz="0 0 0.02" rpy="0 0 0"/>
-  </xacro:iiwa7>
-  <!-- Here we insert a Schunk gripper in the scene -->
-  <xacro:egl90 parent="$(arg robot_name)_link_ee" prefix="$(arg robot_name)_" />
-  <!-- TCP link -->
-  <joint name="gripper_ee_joint" type="fixed">
-    <parent link="$(arg robot_name)_link_ee" />
-    <child link="$(arg robot_name)_gripper_link_ee" />
-    <origin xyz="0 0 0.248" rpy="0 0 0"/>
-  </joint>
-  <link name="$(arg robot_name)_gripper_link_ee"/>
-  <joint name="profile_cams_joint" type="fixed">
-    <parent link="world" />
-    <child link="profile_cams" />
-    <origin xyz="0 0 0" rpy="0 0 0"/>
-  </joint>
-  <link name="profile_cams">
-    <inertial>
-       <origin xyz="0 0 0" rpy="0 0 0"/>
-       <mass value="0.1"/>
-       <inertia ixx="0.0001" ixy="0" ixz="0" iyy="0.0002" iyz="0" izz="0.0001"/>
-    </inertial>
-    <visual>
-      <origin xyz="0 0 0" rpy="0 0 ${90 * pi / 180}"/>
-      <geometry>
-        <mesh filename="package://rll_description/meshes/rll/visual/profile_cams.dae"/>
-      </geometry>
-    </visual>
-    <collision>
-      <origin xyz="0.58 0.82 0.17" rpy="0 0 0"/>
-      <geometry>
-        <box size="0.05 0.05 2.0"/>
-      </geometry>
-    </collision>
-  </link>
-  <!-- Roboception camera -->
-  <xacro:rc_160 parent="profile_cams" prefix="$(arg robot_name)_">
-    <origin xyz="0.577 0.8 0.825" rpy="0 ${180 * pi / 180} 0"/>
-  </xacro:rc_160>
-  <!-- Axis camera -->
-  <joint name="axis_cam_base_joint" type="fixed">
-    <parent link="profile_cams" />
-    <child link="axis_cam_base" />
-    <origin xyz="0.577 0.8 1.137" rpy="${90 * pi / 180} 0 0"/>
-  </joint>
-  <link name="axis_cam_base">
-    <visual>
-      <origin xyz="0 0 0" rpy="0 0 0"/>
-      <geometry>
-        <mesh filename="package://rll_description/meshes/rll/visual/axis_cam_bottom.dae"/>
-      </geometry>
-    </visual>
-    <collision>
-      <origin xyz="0 0 0.035" rpy="0 0 0"/>
-      <geometry>
-        <box size="0.07 0.07 0.07"/>
-      </geometry>
-    </collision>
-  </link>
-  <joint name="axis_cam_top_joint" type="fixed">
-    <parent link="axis_cam_base" />
-    <child link="axis_cam_top" />
-    <origin xyz="0 0 0.068" rpy="${30 * pi / 180} ${30 * pi / 180} ${-65 * pi / 180}"/>
-  </joint>
-  <link name="axis_cam_top">
-    <visual>
-      <origin xyz="0 0 0" rpy="0 0 0"/>
-      <geometry>
-        <mesh filename="package://rll_description/meshes/rll/visual/axis_cam_top.dae"/>
-      </geometry>
-    </visual>
-    <collision>
-      <origin xyz="0 0.01 0.03" rpy="0 0 0"/>
-      <geometry>
-        <box size="0.06 0.11 0.06"/>
-      </geometry>
-    </collision>
-  </link>
-  <!--Extensions -->
-  <xacro:rll_virtual />
-  <xacro:rll_gazebo robot_name="$(arg robot_name)" />
-  <xacro:rll_transmission hardware_interface="$(arg hardware_interface)" robot_name="$(arg robot_name)"/>
+    <xacro:rll_cell hardware_interface="$(arg hardware_interface)" robot_name="$(arg robot_name)"/>
 </robot>

Commit message: description: enable grasp plugin
Signed-off-by: Wolfgang Wiedmeyer <wolfgang.wiedmeyer@kit.edu>

File: rll_description/urdf/rll.gazebo.xacro (robot description, xacro)
@@ -2,17 +2,43 @@
 <robot xmlns:xacro="http://www.ros.org/wiki/xacro">
   <xacro:macro name="rll_gazebo" params="robot_name">
-  <!-- Link Table -->
-  <gazebo reference="table">
-    <mu1>1.0</mu1>
-    <mu2>1.0</mu2>
-    <static>true</static>
-  </gazebo>
-  <gazebo reference="$(arg robot_name)_link_0">
-    <static>true</static>
-  </gazebo>
-  <!-- Link profile_cams -->
-  <gazebo reference="profile_cams">
-    <static>true</static>
-  </gazebo>
+    <!-- Link Table -->
+    <gazebo reference="table">
+      <mu1>1.0</mu1>
+      <mu2>1.0</mu2>
+      <static>true</static>
+    </gazebo>
+    <gazebo reference="$(arg robot_name)_link_0">
+      <static>true</static>
+    </gazebo>
+    <gazebo reference="$(arg robot_name)_gripper_waggon_right">
+      <mu1>1.0</mu1>
+      <mu2>1.0</mu2>
+    </gazebo>
+    <gazebo reference="$(arg robot_name)_gripper_waggon_left">
+      <mu1>1.0</mu1>
+      <mu2>1.0</mu2>
+    </gazebo>
+    <!-- Link profile_cams -->
+    <gazebo reference="profile_cams">
+      <static>true</static>
+    </gazebo>
+    <!-- grasp plugin -->
+    <gazebo>
+      <plugin name="gazebo_grasp_fix" filename="libgazebo_grasp_fix.so">
+        <arm>
+          <arm_name>$(arg robot_name)</arm_name>
+          <palm_link>$(arg robot_name)_link_7</palm_link>
+          <gripper_link>$(arg robot_name)_gripper_waggon_right</gripper_link>
+          <gripper_link>$(arg robot_name)_gripper_waggon_left</gripper_link>
+        </arm>
+        <forces_angle_tolerance>100</forces_angle_tolerance>
+        <update_rate>30</update_rate>
+        <grip_count_threshold>4</grip_count_threshold>
+        <max_grip_count>8</max_grip_count>
+        <release_tolerance>0.0005</release_tolerance>
+        <disable_collisions_on_attach>false</disable_collisions_on_attach>
+        <contact_topic>__default_topic__</contact_topic>
+      </plugin>
+    </gazebo>
   </xacro:macro>
 </robot>

File: rll_description/urdf/rll_cell.xacro (robot description, xacro)
@@ -20,6 +20,6 @@
       <inertial>
         <origin xyz="0 0 0" rpy="0 0 0"/>
-        <mass value="0.1"/>
-        <inertia ixx="0.0001" ixy="0" ixz="0" iyy="0.0002" iyz="0" izz="0.0001"/>
+        <mass value="600"/>
+        <inertia ixx="1" ixy="0" ixz="0" iyy="1" iyz="0" izz="1"/>
       </inertial>
       <visual>
@@ -58,5 +58,4 @@
       </collision>
     </link>
-    <!-- Here we insert an iiwa7 robot in the scene, it's origin is on top of the adapter. -->
     <xacro:iiwa7 hardware_interface="$(arg hardware_interface)" robot_name="$(arg robot_name)" parent="$(arg robot_name)_base_adapter">
       <origin xyz="0 0 0.02" rpy="0 0 0"/>

Commit message: description: check collisions with table and the camera mount in Gazebo
Signed-off-by: Wolfgang Wiedmeyer <wolfgang.wiedmeyer@kit.edu>

File: rll_description/urdf/rll.gazebo.xacro (robot description, xacro)
@@ -6,4 +6,17 @@
       <mu1>10.0</mu1>
       <mu2>10.0</mu2>
+      <selfCollide>true</selfCollide>
+    </gazebo>
+    <!-- profile_cams link includes the cameras in Gazebo -->
+    <!-- These settings ensure that the collision object has maximum stiffness -->
+    <!-- and collisions are immediately detected -->
+    <gazebo reference="profile_cams">
+      <mu1>10.0</mu1>
+      <mu2>10.0</mu2>
+      <selfCollide>true</selfCollide>
+      <maxVel>0.0</maxVel>
+      <minDepth>0.0</minDepth>
+      <kp>1000000.0</kp>
+      <kd>1.0</kd>
     </gazebo>
   </xacro:macro>

File: rll_description/urdf/rll_cell.xacro (robot description, xacro)
@@ -66,7 +66,7 @@
     <link name="profile_cams">
       <inertial>
-        <origin xyz="0 0 0" rpy="0 0 0"/>
-        <mass value="0.1"/>
-        <inertia ixx="0.0001" ixy="0" ixz="0" iyy="0.0002" iyz="0" izz="0.0001"/>
+        <origin xyz="0.58 0.82 0.17" rpy="0 0 0"/>
+        <mass value="5"/>
+        <inertia ixx="1.67" ixy="0" ixz="0" iyy="1.67" iyz="0" izz="0.002"/>
       </inertial>
       <visual>

Commit message: description: add virtual walls to Gazebo model and fix link chain
The virtual walls were missing inertia properties. The xacro is also
cleaned up and uses properties now.

Several links (profile_cams, virtual walls) were directly attached to the
world link which Gazebo doesn't like at all and the Gui crashes when
trying to view the link properties. These links need to be attached to the
table, then Gazebo also correctly puts everything together into one fixed
table link.

Signed-off-by: Wolfgang Wiedmeyer <wolfgang.wiedmeyer@kit.edu>

File: rll_description/urdf/rll.gazebo.xacro (robot description, xacro)
@@ -8,16 +8,4 @@
       <selfCollide>true</selfCollide>
     </gazebo>
-    <!-- profile_cams link includes the cameras in Gazebo -->
-    <!-- These settings ensure that the collision object has maximum stiffness -->
-    <!-- and collisions are immediately detected -->
-    <gazebo reference="profile_cams">
-      <mu1>10.0</mu1>
-      <mu2>10.0</mu2>
-      <selfCollide>true</selfCollide>
-      <maxVel>0.0</maxVel>
-      <minDepth>0.0</minDepth>
-      <kp>1000000.0</kp>
-      <kd>1.0</kd>
-    </gazebo>
   </xacro:macro>
 </robot>

File: rll_description/urdf/rll_cell.xacro (robot description, xacro)
@@ -36,5 +36,5 @@
     </link>
     <joint name="base_adapter_joint" type="fixed">
-      <parent link="world" />
+      <parent link="table" />
       <child link="$(arg robot_name)_base_adapter" />
       <origin xyz="-0.2 0 0" rpy="0 0 0"/>
@@ -60,5 +60,5 @@
     <xacro:egl90 parent="$(arg robot_name)_link_ee" prefix="$(arg robot_name)_" />
     <joint name="profile_cams_joint" type="fixed">
-      <parent link="world" />
+      <parent link="table" />
       <child link="profile_cams" />
       <origin xyz="0 0 0" rpy="0 0 0"/>

File: rll_description/urdf/rll_virtual.xacro (robot description, xacro)
@@ -4,58 +4,89 @@
     <!-- virtual walls -->
     <joint name="wall_joint1" type="fixed">
-      <parent link="world" />
+      <parent link="table" />
       <child link="wall_front" />
-      <origin xyz="0.605 0 0.7" rpy="0 0 0"/>
+      <origin xyz="${wall_origin_x_long_side} 0 ${wall_origin_z}" rpy="0 0 0"/>
     </joint>
     <joint name="wall_joint2" type="fixed">
-      <parent link="world" />
+      <parent link="table" />
       <child link="wall_back" />
-      <origin xyz="-0.605 0 0.7" rpy="0 0 0"/>
+      <origin xyz="-${wall_origin_x_long_side} 0 ${wall_origin_z}" rpy="0 0 0"/>
     </joint>
     <joint name="wall_joint3" type="fixed">
-      <parent link="world" />
+      <parent link="table" />
       <child link="wall_left" />
-      <origin xyz="0 -0.805 0.7" rpy="0 0 0"/>
+      <origin xyz="0 -${wall_origin_y_short_side} ${wall_origin_z}" rpy="0 0 0"/>
     </joint>
     <joint name="wall_joint4" type="fixed">
-      <parent link="world" />
+      <parent link="table" />
       <child link="wall_right" />
-      <origin xyz="0 0.805 0.7" rpy="0 0 0"/>
+      <origin xyz="0 ${wall_origin_y_short_side} ${wall_origin_z}" rpy="0 0 0"/>
     </joint>
     <link name="wall_front">
+      <inertial>
+          <xacro:insert_block name="wall_inertia_long_side" />
+      </inertial>
       <collision>
         <origin xyz="0 0 0" rpy="0 0 0"/>
         <geometry>
-          <box size="0.01 1.6 1.4" rpy="0 0 0"/>
+          <xacro:insert_block name="collision_geometry_wall_long_side" />
         </geometry>
       </collision>
     </link>
     <link name="wall_back">
+      <inertial>
+          <xacro:insert_block name="wall_inertia_long_side" />
+      </inertial>
       <collision>
         <origin xyz="0 0 0" rpy="0 0 0"/>
         <geometry>
-          <box size="0.01 1.6 1.4" rpy="0 0 0"/>
+          <xacro:insert_block name="collision_geometry_wall_long_side" />
         </geometry>
       </collision>
     </link>
     <link name="wall_left">
+      <inertial>
+          <xacro:insert_block name="wall_inertia_short_side" />
+      </inertial>
       <collision>
         <origin xyz="0 0 0" rpy="0 0 0"/>
         <geometry>
-          <box size="1.2 0.01 1.4" rpy="0 0 0"/>
+          <xacro:insert_block name="collision_geometry_wall_short_side" />
         </geometry>
       </collision>
     </link>
     <link name="wall_right">
+      <inertial>
+          <xacro:insert_block name="wall_inertia_short_side" />
+      </inertial>
       <collision>
         <origin xyz="0 0 0" rpy="0 0 0"/>
         <geometry>
-          <box size="1.2 0.01 1.4" rpy="0 0 0"/>
+          <xacro:insert_block name="collision_geometry_wall_short_side" />
         </geometry>
       </collision>
     </link>
-      <material name="transparent">
-        <color rgba="0.8784 0.8745 0.8588 0.3"/>
-      </material>
+    <material name="transparent">
+      <color rgba="0.8784 0.8745 0.8588 0.3"/>
+    </material>
   </xacro:macro>
+  <xacro:property name="wall_origin_x_long_side" value="0.605" />
+  <xacro:property name="wall_origin_y_short_side" value="0.805" />
+  <xacro:property name="wall_origin_z" value="0.7" />
+  <xacro:property name="collision_geometry_wall_long_side">
+    <box size="0.01 1.6 1.4" rpy="0 0 0"/>
+  </xacro:property>
+  <xacro:property name="collision_geometry_wall_short_side">
+    <box size="1.2 0.01 1.4" rpy="0 0 0"/>
+  </xacro:property>
+  <xacro:property name="wall_inertia_long_side">
+      <origin xyz="0 0 0" rpy="0 0 0"/>
+      <mass value="5"/>
+      <inertia ixx="1.88" ixy="0" ixz="0" iyy="0.82" iyz="0" izz="1.07"/>
+  </xacro:property>
+  <xacro:property name="wall_inertia_short_side">
+      <origin xyz="0 0 0" rpy="0 0 0"/>
+      <mass value="4"/>
+      <inertia ixx="0.65" ixy="0" ixz="0" iyy="1.13" iyz="0" izz="0.48"/>
+  </xacro:property>
 </robot>
