Commit message: Rename roboception camera frame
This is now the uncalibrated one. The calibrated one will be published
by the driver.

Signed-off-by: Wolfgang Wiedmeyer <wolfgang.wiedmeyer@kit.edu>

File: rll_description/urdf/visard160/rc_visard_160.xacro (robot description, xacro)
@@ -36,8 +36,8 @@
     <joint name="${prefix}roboception_camera" type="fixed">
       <parent link="${prefix}roboception_adapter"/>
-      <child link="${prefix}roboception_camera"/>
+      <child link="${prefix}roboception_camera_uncal"/>
       <origin xyz="-0.031 0.0375 0.08" rpy="${-45 * pi / 180} ${90 * pi / 180} ${180 * pi / 180}"/>
     </joint>
-    <link name="${prefix}roboception_camera">
+    <link name="${prefix}roboception_camera_uncal">
       <visual>
         <geometry>
