Commit message: gripper movable in simulation
Signed-off-by: Wolfgang Wiedmeyer <wolfgang.wiedmeyer@kit.edu>

File: rll_description/urdf/egl90/egl90_macro.xacro (robot description, xacro)
@@ -9,6 +9,8 @@
   <xacro:property name="jaw_base_y" value="0.0228"/>
   <xacro:property name="jaw_base_z" value="0.0191"/>
+  <xacro:property name="finger_mass" value="0.1" />
+  <xacro:property name="gripper_mass" value="0.3" />
   <xacro:macro name="egl90-jaws" params="prefix x min max *mesh">
-    <joint name="egl_position" type="fixed">
+    <joint name="egl_position" type="prismatic">
       <parent link="${prefix}jaw_base"/>
       <child link="${prefix}finger_right"/>
@@ -18,4 +20,9 @@
     </joint>
     <link name="${prefix}finger_right">
+      <inertial>
+        <origin xyz="0 0 0" rpy="0 0 0"/>
+        <mass value="${finger_mass}"/>
+        <inertia ixx="0.002" ixy="0" ixz="0" iyy="0.0002" iyz="0" izz="0.0002"/>
+      </inertial>
       <visual>
         <origin xyz="0 0 0" rpy="${90 * PI / 180} 0 ${90 * PI / 180}"/>
@@ -34,5 +41,5 @@
       </collision>
     </link>
-    <joint name="egl_position_mimic" type="fixed">
+    <joint name="egl_position_mimic" type="prismatic">
       <parent link="${prefix}jaw_base"/>
       <child link="${prefix}finger_left"/>
@@ -40,7 +47,11 @@
       <axis xyz="1 0 0"/>
       <limit effort="100.0" lower="${min}" upper="${max}" velocity="100.0"/>
-      <mimic joint="egl_position" multiplier="1"/>
     </joint>
     <link name="${prefix}finger_left">
+      <inertial>
+        <origin xyz="0 0 0" rpy="0 0 0"/>
+        <mass value="${finger_mass}"/>
+        <inertia ixx="0.002" ixy="0" ixz="0" iyy="0.0002" iyz="0" izz="0.0002"/>
+      </inertial>
       <visual>
         <origin xyz="0 0 0" rpy="${90 * PI / 180} 0 ${90 * PI / 180}"/>
@@ -94,4 +105,9 @@
     </joint>
     <link name="${prefix}jaw_base">
+      <inertial>
+        <origin xyz="0 0 0" rpy="0 0 0"/>
+        <mass value="${gripper_mass}"/>
+        <inertia ixx="0.0001" ixy="0" ixz="0" iyy="0.0002" iyz="0" izz="0.0001"/>
+      </inertial>
       <visual>
         <origin rpy="0 0 0" xyz="0 0 ${-jaw_base_z/2}"/>

File: rll_description/urdf/rll_setup.urdf.xacro (robot description, xacro)
@@ -196,4 +196,26 @@
   </joint>
   <link name="$(arg robot_name)_gripper_link_ee"/>
+  <!-- gripper transmissions -->
+  <transmission name="$(arg robot_name)_tran_8">
+    <type>transmission_interface/SimpleTransmission</type>
+    <joint name="egl_position">
+      <hardwareInterface>hardware_interface/EffortJointInterface</hardwareInterface>
+    </joint>
+    <actuator name="$(arg robot_name)_motor_8">
+      <hardwareInterface>hardware_interface/EffortJointInterface</hardwareInterface>
+      <mechanicalReduction>1</mechanicalReduction>
+    </actuator>
+  </transmission>
+  <transmission name="$(arg robot_name)_tran_9">
+    <type>transmission_interface/SimpleTransmission</type>
+    <joint name="egl_position_mimic">
+      <hardwareInterface>hardware_interface/EffortJointInterface</hardwareInterface>
+    </joint>
+    <actuator name="$(arg robot_name)_motor_9">
+      <hardwareInterface>hardware_interface/EffortJointInterface</hardwareInterface>
+      <mechanicalReduction>1</mechanicalReduction>
+    </actuator>
+  </transmission>
+  <!-- Roboception camera -->
   <joint name="roboception_base_joint" type="fixed">
     <parent link="world" />

Commit message: description: cleanup
Signed-off-by: Wolfgang Wiedmeyer <wolfgang.wiedmeyer@kit.edu>

File: rll_description/urdf/egl90/egl90_macro.xacro (robot description, xacro)
@@ -30,7 +30,4 @@
           <xacro:insert_block name="mesh"/>
         </geometry>
-        <material name="black ">
-          <color rgba="1.0 1.0 1.0 1.0"/>
-        </material>
       </visual>
       <collision>
@@ -59,7 +56,4 @@
           <xacro:insert_block name="mesh"/>
         </geometry>
-        <material name="black ">
-          <color rgba="1.0 1.0 1.0 1.0"/>
-        </material>
       </visual>
       <collision>

File: rll_description/urdf/rll_setup.urdf.xacro (robot description, xacro)
@@ -110,19 +110,4 @@
     </collision>
   </link>
-  <gazebo reference="world">
-    <static>true</static>
-  </gazebo>
-  <gazebo reference="wall_front">
-    <static>true</static>
-  </gazebo>
-  <gazebo reference="wall_back">
-    <static>true</static>
-  </gazebo>
-  <gazebo reference="wall_left">
-    <static>true</static>
-  </gazebo>
-  <gazebo reference="wall_right">
-    <static>true</static>
-  </gazebo>
   <joint name="base_adapter_joint" type="fixed">
     <parent link="world" />
@@ -240,4 +225,8 @@
     </collision>
   </link>
+  <gazebo reference="$(arg robot_name)_base_adapter">
+    <material>Gazebo/Grey</material>
+    <static>true</static>
+  </gazebo>
   <material name="steel">
     <color rgba="0.8784 0.8745 0.8588 1.0"/>

Commit message: WIP: description: rework gripper
Signed-off-by: Wolfgang Wiedmeyer <wolfgang.wiedmeyer@kit.edu>

File: rll_description/urdf/egl90/egl90_macro.xacro (robot description, xacro)
@@ -1,23 +1,40 @@
 <?xml version="1.0"?>
 <robot name="egl90" xmlns:xacro="http://www.ros.org/wiki/xacro">
-  <material name="egl90-metal">
-    <color rgba="0.5 0.45 0.4 1"/>
-  </material>
-  <xacro:property name="base_x" value="0.112"/>
-  <xacro:property name="base_y" value="0.090"/>
-  <xacro:property name="base_z" value="0.08725"/>
-  <xacro:property name="jaw_base_y" value="0.0228"/>
-  <xacro:property name="jaw_base_z" value="0.0191"/>
   <xacro:property name="finger_mass" value="0.1" />
-  <xacro:property name="gripper_mass" value="0.3" />
-  <xacro:macro name="egl90-jaws" params="prefix x min max *mesh">
+  <xacro:macro name="egl90" params="parent prefix *origin">
+    <joint name="${prefix}mount" type="fixed">
+      <xacro:insert_block name="origin"/>
+      <parent link="${parent}"/>
+      <child link="${prefix}gripper_base"/>
+    </joint>
+    <link name="${prefix}gripper_base">
+      <inertial>
+        <origin xyz="0.055 0 0" rpy="${pi/2} 0 ${pi/2}"/>
+        <mass value="0.3"/>
+        <inertia ixx="0.0001" ixy="0" ixz="0" iyy="0.0002" iyz="0" izz="0.0001"/>
+      </inertial>
+      <visual>
+        <origin xyz="0 0 0" rpy="0 0 0" />
+        <geometry>
+          <mesh filename="package://rll_description/meshes/egl90/visual/gripper_base.stl" scale="0.001 0.001 0.001"/>
+        </geometry>
+      </visual>
+      <collision>
+        <origin xyz="0 0.059 -0.025" rpy="0 0 0"/>
+        <geometry>
+          <box size="0.09 0.108 0.18"/>
+        </geometry>
+      </collision>
+    </link>
+  </xacro:macro>
+  <xacro:macro name="egl90-jaws" params="prefix min max *mesh">
     <joint name="egl_position" type="prismatic">
-      <parent link="${prefix}jaw_base"/>
-      <child link="${prefix}finger_right"/>
-      <origin rpy="0.0 0.0 ${pi}" xyz="${x - 0.1} -0.013 0.005"/>
+      <parent link="${prefix}gripper_base"/>
+      <child link="${prefix}gripper_finger_right"/>
+      <origin xyz="-0.013 0.1063 -0.1" rpy="0 ${pi} 0"/>
       <axis xyz="1 0 0"/>
       <limit effort="100.0" lower="${min}" upper="${max}" velocity="100.0"/>
     </joint>
-    <link name="${prefix}finger_right">
+    <link name="${prefix}gripper_finger_right">
       <inertial>
         <origin xyz="0 0 0" rpy="0 0 0"/>
@@ -26,5 +43,5 @@
       </inertial>
       <visual>
-        <origin xyz="0 0 0" rpy="${90 * PI / 180} 0 ${90 * PI / 180}"/>
+        <origin xyz="0 0 0" rpy="0 0 0"/>
         <geometry>
           <xacro:insert_block name="mesh"/>
@@ -32,5 +49,5 @@
       </visual>
       <collision>
-        <origin xyz="0 0 0" rpy="${90 * PI / 180} 0 ${90 * PI / 180}"/>
+        <origin xyz="0 0 0" rpy="0 0 0"/>
         <geometry>
           <xacro:insert_block name="mesh"/>
@@ -39,11 +56,11 @@
     </link>
     <joint name="egl_position_mimic" type="prismatic">
-      <parent link="${prefix}jaw_base"/>
-      <child link="${prefix}finger_left"/>
-      <origin rpy="0.0 0.0 0.0" xyz="${x + 0.1} 0.013 0.005"/>
+      <parent link="${prefix}gripper_base"/>
+      <child link="${prefix}gripper_finger_left"/>
+      <origin xyz="0.013 0.1063 -0.02" rpy="0 0 0"/>
       <axis xyz="1 0 0"/>
       <limit effort="100.0" lower="${min}" upper="${max}" velocity="100.0"/>
     </joint>
-    <link name="${prefix}finger_left">
+    <link name="${prefix}gripper_finger_left">
       <inertial>
         <origin xyz="0 0 0" rpy="0 0 0"/>
@@ -52,5 +69,5 @@
       </inertial>
       <visual>
-        <origin xyz="0 0 0" rpy="${90 * PI / 180} 0 ${90 * PI / 180}"/>
+        <origin xyz="0 0 0" rpy="0 0 0"/>
         <geometry>
           <xacro:insert_block name="mesh"/>
@@ -58,5 +75,5 @@
       </visual>
       <collision>
-        <origin xyz="0 0 0" rpy="${90 * PI / 180} 0 ${90 * PI / 180}"/>
+        <origin xyz="0 0 0" rpy="0 0 0"/>
         <geometry>
           <xacro:insert_block name="mesh"/>
@@ -65,51 +82,3 @@
     </link>
   </xacro:macro>
-  <!-- Added to figure out orientation -->
-  <xacro:macro name="egl90-connector" params="y z">
-    <visual>
-      <origin rpy="0 1.5708 0" xyz="${-base_x/2 - 0.005} ${y} ${base_z/2 + z}"/>
-      <geometry>
-        <cylinder length="0.01" radius="0.005"/>
-      </geometry>
-      <material name="egl90-metal"/>
-    </visual>
-  </xacro:macro>
-  <xacro:macro name="egl90" params="parent prefix *origin">
-    <joint name="${prefix}mount" type="fixed">
-      <xacro:insert_block name="origin"/>
-      <parent link="${parent}"/>
-      <child link="${prefix}base"/>
-    </joint>
-    <link name="${prefix}base">
-      <visual>
-        <origin rpy="0 0 0" xyz="0 0 ${base_z/2}"/>
-        <geometry>
-          <box size="${base_x} ${base_y} ${base_z}"/>
-        </geometry>
-        <material name="egl90-metal"/>
-      </visual>
-      <xacro:egl90-connector y="-0.02" z="0.02"/>
-      <xacro:egl90-connector y="-0.02" z="-0.02"/>
-      <xacro:egl90-connector y="0.02" z="-0.02"/>
-    </link>
-    <joint name="${prefix}jaw_mount" type="fixed">
-      <origin rpy="0 0 0" xyz="0 0 ${base_z + jaw_base_z}"/>
-      <parent link="${prefix}base"/>
-      <child link="${prefix}jaw_base"/>
-    </joint>
-    <link name="${prefix}jaw_base">
-      <inertial>
-        <origin xyz="0 0 0" rpy="0 0 0"/>
-        <mass value="${gripper_mass}"/>
-        <inertia ixx="0.0001" ixy="0" ixz="0" iyy="0.0002" iyz="0" izz="0.0001"/>
-      </inertial>
-      <visual>
-        <origin rpy="0 0 0" xyz="0 0 ${-jaw_base_z/2}"/>
-        <geometry>
-          <box size="${base_x} ${jaw_base_y} ${jaw_base_z}"/>
-        </geometry>
-        <material name="egl90-metal"/>
-      </visual>
-    </link>
-  </xacro:macro>
 </robot>

File: rll_description/urdf/rll_setup.urdf.xacro (robot description, xacro)
@@ -136,9 +136,9 @@
     <parent link="$(arg robot_name)_link_ee" />
     <child link="$(arg robot_name)_gripper_adapter" />
-    <origin xyz="0 0 0" rpy="0 0 0"/>
+    <origin xyz="0 0 0.024" rpy="0 0 0"/>
   </joint>
   <link name="$(arg robot_name)_gripper_adapter">
     <visual>
-      <origin xyz="0 0 0.024" rpy="${180 * PI / 180} 0 ${-90 * PI / 180}"/>
+      <origin xyz="0 0 0" rpy="${180 * PI / 180} 0 ${-90 * PI / 180}"/>
       <geometry>
         <mesh filename="package://rll_description/meshes/egl90/visual/gripper_adapter.dae" scale="0.001 0.001 0.001"/>
@@ -146,5 +146,5 @@
     </visual>
     <collision>
-      <origin xyz="0 0 0.024" rpy="${180 * PI / 180} 0 ${-90 * PI / 180}"/>
+      <origin xyz="0 0 0" rpy="${180 * PI / 180} 0 ${-90 * PI / 180}"/>
       <geometry>
         <mesh filename="package://rll_description/meshes/egl90/visual/gripper_adapter.dae" scale="0.001 0.001 0.001"/>
@@ -153,7 +153,7 @@
   </link>
   <xacro:egl90 parent="$(arg robot_name)_gripper_adapter" prefix="$(arg robot_name)_">
-    <origin xyz="0 0 0.024" rpy="0 0 ${-90 * PI / 180}"/>
+    <origin xyz="0 0.055 0" rpy="${90 * PI / 180} 0 ${180 * PI / 180}"/>
   </xacro:egl90>
-  <xacro:egl90-jaws prefix="$(arg robot_name)_" x="0.0" min="-0.015" max="0.026">
+  <xacro:egl90-jaws prefix="$(arg robot_name)_" min="-0.015" max="0.026">
     <mesh filename="package://rll_description/meshes/egl90/visual/gripper_finger.dae" scale="0.001 0.001 0.001"/>
   </xacro:egl90-jaws>
@@ -247,7 +247,4 @@
     <static>true</static>
   </gazebo>
-  <gazebo reference="$(arg robot_name)_gripper_adapter">
-    <static>true</static>
-  </gazebo>
   <material name="transparent">
     <color rgba="0.8784 0.8745 0.8588 0.3"/>

File: rll_description/urdf/visard160/rc_visard_160.xacro (robot description, xacro)
@@ -2,10 +2,10 @@
 <robot name="rc_visard_160" xmlns:xacro="http://www.ros.org/wiki/xacro">
   <xacro:macro name="rc_160" params="prefix parent *origin">
-    <joint name="${prefix}camera" type="fixed">
+    <joint name="${prefix}roboception_camera" type="fixed">
       <parent link="${parent}"/>
-      <child link="${prefix}camera"/>
+      <child link="${prefix}roboception_camera"/>
       <xacro:insert_block name="origin"/>
     </joint>
-    <link name="${prefix}camera">
+    <link name="${prefix}roboception_camera">
       <visual>
           <geometry>
@@ -20,8 +20,8 @@
       </collision>
     </link>
-  <link name="${prefix}mounting"/>
+  <link name="${prefix}roboception_mounting"/>
   <joint name="${prefix}mounting_to_camera" type="fixed">
-    <parent link="${prefix}camera"/>
-    <child link="${prefix}mounting"/>
+    <parent link="${prefix}roboception_camera"/>
+    <child link="${prefix}roboception_mounting"/>
     <origin xyz="0.080 0.0375 -0.031" />
   </joint>

Commit message: WIP: description: reorganize and small fixes
Signed-off-by: Wolfgang Wiedmeyer <wolfgang.wiedmeyer@kit.edu>

File: rll_description/urdf/egl90/egl90_macro.xacro (robot description, xacro)
@@ -3,12 +3,31 @@
   <xacro:property name="finger_mass" value="0.1" />
   <xacro:macro name="egl90" params="parent prefix *origin">
+    <joint name="gripper_adapter_joint" type="fixed">
+      <parent link="${parent}" />
+      <child link="${prefix}gripper_adapter" />
+      <xacro:insert_block name="origin"/>
+    </joint>
+    <link name="${prefix}gripper_adapter">
+      <visual>
+        <origin xyz="0 0 0" rpy="${180 * PI / 180} 0 ${-90 * PI / 180}"/>
+        <geometry>
+          <mesh filename="package://rll_description/meshes/egl90/visual/gripper_adapter.dae" scale="0.001 0.001 0.001"/>
+        </geometry>
+      </visual>
+      <collision>
+        <origin xyz="0 0 -0.015" rpy="${180 * PI / 180} 0 ${-90 * PI / 180}"/>
+        <geometry>
+          <box size="0.09 0.07 0.03"/>
+        </geometry>
+      </collision>
+    </link>
     <joint name="${prefix}mount" type="fixed">
-      <xacro:insert_block name="origin"/>
-      <parent link="${parent}"/>
+      <parent link="${prefix}gripper_adapter"/>
       <child link="${prefix}gripper_base"/>
+      <origin xyz="0 0.055 0" rpy="${90 * PI / 180} 0 ${180 * PI / 180}"/>
     </joint>
     <link name="${prefix}gripper_base">
       <inertial>
-        <origin xyz="0.055 0 0" rpy="${pi/2} 0 ${pi/2}"/>
+        <origin xyz="0.055 0 0" rpy="${90 * PI / 180} 0 ${90 * PI / 180}"/>
         <mass value="0.3"/>
         <inertia ixx="0.0001" ixy="0" ixz="0" iyy="0.0002" iyz="0" izz="0.0001"/>
@@ -21,5 +40,5 @@
       </visual>
       <collision>
-        <origin xyz="0 0.059 -0.025" rpy="0 0 0"/>
+        <origin xyz="0 0.055 -0.025" rpy="0 0 0"/>
         <geometry>
           <box size="0.09 0.108 0.18"/>
@@ -32,5 +51,5 @@
       <parent link="${prefix}gripper_base"/>
       <child link="${prefix}gripper_finger_right"/>
-      <origin xyz="-0.013 0.1063 -0.1" rpy="0 ${pi} 0"/>
+      <origin xyz="-0.013 0.1063 -0.1" rpy="0 ${180 * PI / 180} 0"/>
       <axis xyz="1 0 0"/>
       <limit effort="100.0" lower="${min}" upper="${max}" velocity="100.0"/>

File: rll_description/urdf/rll_setup.urdf.xacro (robot description, xacro)
@@ -7,8 +7,4 @@
   <xacro:arg name="hardware_interface" default="PositionJointInterface"/>
   <xacro:arg name="robot_name" default="iiwa"/>
-  <!--  Define the origin of your 3D space
-       Here we define a box lying at 0,0,0 with some dimensions. In reality, our robot is placed on top of a table.
-       This will include the table top in the scene and avoid the robot to hit it when using MoveIt!
-  -->
   <link name="world">
     <visual>
@@ -132,26 +128,7 @@
     <origin xyz="0 0 0.02" rpy="0 0 0"/>
   </xacro:iiwa7>
-  <!-- Here we insert a schunk gripper in the scene -->
-  <joint name="gripper_adapter_joint" type="fixed">
-    <parent link="$(arg robot_name)_link_ee" />
-    <child link="$(arg robot_name)_gripper_adapter" />
+  <!-- Here we insert a Schunk gripper in the scene -->
+  <xacro:egl90 parent="$(arg robot_name)_link_ee" prefix="$(arg robot_name)_">
     <origin xyz="0 0 0.024" rpy="0 0 0"/>
-  </joint>
-  <link name="$(arg robot_name)_gripper_adapter">
-    <visual>
-      <origin xyz="0 0 0" rpy="${180 * PI / 180} 0 ${-90 * PI / 180}"/>
-      <geometry>
-        <mesh filename="package://rll_description/meshes/egl90/visual/gripper_adapter.dae" scale="0.001 0.001 0.001"/>
-      </geometry>
-    </visual>
-    <collision>
-      <origin xyz="0 0 0" rpy="${180 * PI / 180} 0 ${-90 * PI / 180}"/>
-      <geometry>
-        <mesh filename="package://rll_description/meshes/egl90/visual/gripper_adapter.dae" scale="0.001 0.001 0.001"/>
-      </geometry>
-    </collision>
-  </link>
-  <xacro:egl90 parent="$(arg robot_name)_gripper_adapter" prefix="$(arg robot_name)_">
-    <origin xyz="0 0.055 0" rpy="${90 * PI / 180} 0 ${180 * PI / 180}"/>
   </xacro:egl90>
   <xacro:egl90-jaws prefix="$(arg robot_name)_" min="-0.015" max="0.026">
@@ -205,39 +182,7 @@
     </collision>
   </link>
-  <joint name="roboception_gusset_joint" type="fixed">
-    <parent link="profile_cams" />
-    <child link="roboception_gusset" />
+  <!-- Roboception camera -->
+  <xacro:rc_160 parent="profile_cams" prefix="$(arg robot_name)_">
     <origin xyz="0.577 0.8 0.825" rpy="0 ${180 * PI / 180} 0"/>
-  </joint>
-  <link name="roboception_gusset">
-    <visual>
-      <origin xyz="0 0 0" rpy="0 0 0"/>
-      <geometry>
-        <mesh filename="package://rll_description/meshes/rll/visual/roboception_gusset.dae"/>
-      </geometry>
-    </visual>
-    <collision>
-      <origin xyz="0 -0.05 0.05" rpy="0 0 0"/>
-      <geometry>
-        <box size="0.05 0.1 0.1"/>
-      </geometry>
-    </collision>
-  </link>
-  <!-- Roboception camera -->
-  <joint name="roboception_adapter_joint" type="fixed">
-    <parent link="roboception_gusset" />
-    <child link="roboception_adapter" />
-    <origin xyz="0.03 -0.075 0" rpy="${-90 * PI / 180} 0 ${135 * PI / 180}"/>
-  </joint>
-  <link name="roboception_adapter">
-    <visual>
-      <origin xyz="0 0 0" rpy="0 0 0"/>
-      <geometry>
-        <mesh filename="package://rll_description/meshes/rll/visual/roboception_adapter.dae"/>
-      </geometry>
-    </visual>
-  </link>
-  <xacro:rc_160 parent="roboception_adapter" prefix="$(arg robot_name)_">
-    <origin xyz="-0.03 0.03 -0.08" rpy="${45 * PI / 180} ${-90 * PI / 180} 0"/>
   </xacro:rc_160>
   <gazebo reference="world">

File: rll_description/urdf/visard160/rc_visard_160.xacro (robot description, xacro)
@@ -2,28 +2,60 @@
 <robot name="rc_visard_160" xmlns:xacro="http://www.ros.org/wiki/xacro">
   <xacro:macro name="rc_160" params="prefix parent *origin">
+    <joint name="roboception_gusset_joint" type="fixed">
+      <parent link="${parent}" />
+      <child link="${prefix}roboception_gusset" />
+      <xacro:insert_block name="origin"/>
+    </joint>
+    <link name="${prefix}roboception_gusset">
+      <visual>
+        <origin xyz="0 0 0" rpy="0 0 0"/>
+        <geometry>
+          <mesh filename="package://rll_description/meshes/rll/visual/roboception_gusset.dae"/>
+        </geometry>
+      </visual>
+      <collision>
+        <origin xyz="0 -0.05 0.05" rpy="0 0 0"/>
+        <geometry>
+          <box size="0.05 0.1 0.1"/>
+        </geometry>
+      </collision>
+    </link>
+    <joint name="${prefix}roboception_adapter_joint" type="fixed">
+      <parent link="${prefix}roboception_gusset" />
+      <child link="${prefix}roboception_adapter" />
+      <origin xyz="0.03 -0.075 0" rpy="${-90 * PI / 180} 0 ${135 * PI / 180}"/>
+    </joint>
+    <link name="${prefix}roboception_adapter">
+      <visual>
+        <origin xyz="0 0 0" rpy="0 0 0"/>
+        <geometry>
+          <mesh filename="package://rll_description/meshes/rll/visual/roboception_adapter.dae"/>
+        </geometry>
+      </visual>
+    </link>
     <joint name="${prefix}roboception_camera" type="fixed">
-      <parent link="${parent}"/>
+      <parent link="${prefix}roboception_adapter"/>
       <child link="${prefix}roboception_camera"/>
-      <xacro:insert_block name="origin"/>
+      <origin xyz="-0.03 0.03 -0.08" rpy="${45 * PI / 180} ${-90 * PI / 180} 0"/>
     </joint>
     <link name="${prefix}roboception_camera">
       <visual>
-          <geometry>
-              <mesh filename="package://rll_description/meshes/visard160/visual/rc_visard_160.dae"/>
-          </geometry>
+        <geometry>
+          <mesh filename="package://rll_description/meshes/visard160/visual/rc_visard_160.dae"/>
+        </geometry>
       </visual>
       <collision>
-          <origin xyz="0.08 0.03 -0.05" rpy="0 0 0"/>
-          <geometry>
-              <box size="0.27 0.2 0.27"/>
-          </geometry>
+        <origin xyz="0.08 0.03 -0.05" rpy="0 0 0"/>
+        <geometry>
+          <box size="0.27 0.2 0.27"/>
+        </geometry>
       </collision>
     </link>
-  <link name="${prefix}roboception_mounting"/>
-  <joint name="${prefix}mounting_to_camera" type="fixed">
-    <parent link="${prefix}roboception_camera"/>
-    <child link="${prefix}roboception_mounting"/>
-    <origin xyz="0.080 0.0375 -0.031" />
-  </joint>
+    <link name="${prefix}roboception_mounting"/>
+    <joint name="${prefix}mounting_to_camera" type="fixed">
+      <parent link="${prefix}roboception_camera"/>
+      <child link="${prefix}roboception_mounting"/>
+      <origin xyz="0.080 0.0375 -0.031" />
+    </joint>
   </xacro:macro>
-  </robot>
+</robot>
