Commit message: WIP: description and Gazebo: reorganize and major improvements
Thanks to Yutong Wang for helping with this!

Signed-off-by: Wolfgang Wiedmeyer <wolfgang.wiedmeyer@kit.edu>

File: rll_description/urdf/egl90/egl90_macro.xacro (robot description, xacro)
@@ -10,5 +10,5 @@
     <link name="${prefix}gripper_adapter">
       <visual>
-        <origin xyz="0 0 0" rpy="${180 * PI / 180} 0 ${-90 * PI / 180}"/>
+        <origin xyz="0 0 0" rpy="${180 * pi / 180} 0 ${-90 * pi / 180}"/>
         <geometry>
           <mesh filename="package://rll_description/meshes/egl90/visual/gripper_adapter.dae" scale="0.001 0.001 0.001"/>
@@ -16,5 +16,5 @@
       </visual>
       <collision>
-        <origin xyz="0 0 -0.015" rpy="${180 * PI / 180} 0 ${-90 * PI / 180}"/>
+        <origin xyz="0 0 -0.015" rpy="${180 * pi / 180} 0 ${-90 * pi / 180}"/>
         <geometry>
           <box size="0.09 0.07 0.03"/>
@@ -25,9 +25,9 @@
       <parent link="${prefix}gripper_adapter"/>
       <child link="${prefix}gripper_base"/>
-      <origin xyz="0 0.055 0" rpy="${90 * PI / 180} 0 ${180 * PI / 180}"/>
+      <origin xyz="0 0.055 0" rpy="${90 * pi / 180} 0 ${180 * pi / 180}"/>
     </joint>
     <link name="${prefix}gripper_base">
       <inertial>
-        <origin xyz="0.055 0 0" rpy="${90 * PI / 180} 0 ${90 * PI / 180}"/>
+        <origin xyz="0.055 0 0" rpy="${90 * pi / 180} 0 ${90 * pi / 180}"/>
         <mass value="0.3"/>
         <inertia ixx="0.0001" ixy="0" ixz="0" iyy="0.0002" iyz="0" izz="0.0001"/>
@@ -51,5 +51,5 @@
       <parent link="${prefix}gripper_base"/>
       <child link="${prefix}gripper_finger_right"/>
-      <origin xyz="-0.013 0.1063 -0.1" rpy="0 ${180 * PI / 180} 0"/>
+      <origin xyz="-0.013 0.1063 -0.1" rpy="0 ${180 * pi / 180} 0"/>
       <axis xyz="1 0 0"/>
       <limit effort="100.0" lower="${min}" upper="${max}" velocity="100.0"/>

File: rll_description/urdf/iiwa7/iiwa7.xacro (robot description, xacro)
@@ -11,5 +11,4 @@
   <xacro:property name="max_effort" value="300"/>
   <xacro:property name="max_velocity" value="10"/>
-  <xacro:property name="PI" value="3.1415926535897931"/>
   <xacro:macro name="iiwa7" params="parent hardware_interface robot_name *origin">
     <!--joint between {parent} and link_0-->
@@ -48,8 +47,8 @@
       <origin xyz="0 0 0.157" rpy="0 0 0"/>
       <axis xyz="0 0 1"/>
-      <limit lower="${-170 * PI / 180}" upper="${170 * PI / 180}"
-             effort="${max_effort}" velocity="${98 * PI / 180}" />
-      <safety_controller soft_lower_limit="${-168 * PI / 180}"
-                         soft_upper_limit="${168 * PI / 180}"
+      <limit lower="${-170 * pi / 180}" upper="${170 * pi / 180}"
+             effort="${max_effort}" velocity="${98 * pi / 180}" />
+      <safety_controller soft_lower_limit="${-168 * pi / 180}"
+                         soft_upper_limit="${168 * pi / 180}"
                          k_position="${safety_controller_k_pos}"
                          k_velocity="${safety_controller_k_vel}"/>
@@ -78,8 +77,8 @@
       <origin xyz="0 0 0.183" rpy="0 0 0"/>
       <axis xyz="0 1 0"/>
-      <limit lower="${-120 * PI / 180}" upper="${120 * PI / 180}"
-             effort="${max_effort}" velocity="${98 * PI / 180}" />
-      <safety_controller soft_lower_limit="${-118 * PI / 180}"
-                         soft_upper_limit="${118 * PI / 180}"
+      <limit lower="${-120 * pi / 180}" upper="${120 * pi / 180}"
+             effort="${max_effort}" velocity="${98 * pi / 180}" />
+      <safety_controller soft_lower_limit="${-118 * pi / 180}"
+                         soft_upper_limit="${118 * pi / 180}"
                          k_position="${safety_controller_k_pos}"
                          k_velocity="${safety_controller_k_vel}"/>
@@ -108,8 +107,8 @@
       <origin xyz="0 0 0.185" rpy="0 0 0"/>
       <axis xyz="0 0 1"/>
-      <limit lower="${-170 * PI / 180}" upper="${170 * PI / 180}"
-             effort="${max_effort}" velocity="${100 * PI / 180}" />
-      <safety_controller soft_lower_limit="${-168 * PI / 180}"
-                         soft_upper_limit="${168 * PI / 180}"
+      <limit lower="${-170 * pi / 180}" upper="${170 * pi / 180}"
+             effort="${max_effort}" velocity="${100 * pi / 180}" />
+      <safety_controller soft_lower_limit="${-168 * pi / 180}"
+                         soft_upper_limit="${168 * pi / 180}"
                          k_position="${safety_controller_k_pos}"
                          k_velocity="${safety_controller_k_vel}"/>
@@ -138,8 +137,8 @@
       <origin xyz="0 0 0.215" rpy="0 0 0"/>
       <axis xyz="0 -1 0"/>
-      <limit lower="${-120 * PI / 180}" upper="${120 * PI / 180}"
-             effort="${max_effort}" velocity="${130 * PI / 180}" />
-      <safety_controller soft_lower_limit="${-118 * PI / 180}"
-                         soft_upper_limit="${118 * PI / 180}"
+      <limit lower="${-120 * pi / 180}" upper="${120 * pi / 180}"
+             effort="${max_effort}" velocity="${130 * pi / 180}" />
+      <safety_controller soft_lower_limit="${-118 * pi / 180}"
+                         soft_upper_limit="${118 * pi / 180}"
                          k_position="${safety_controller_k_pos}"
                          k_velocity="${safety_controller_k_vel}"/>
@@ -168,8 +167,8 @@
       <origin xyz="0 0 0.4" rpy="0 0 0"/>
       <axis xyz="0 0 1"/>
-      <limit lower="${-170 * PI / 180}" upper="${170 * PI / 180}"
-             effort="${max_effort}" velocity="${140 * PI / 180}" />
-      <safety_controller soft_lower_limit="${-168 * PI / 180}"
-                         soft_upper_limit="${168 * PI / 180}"
+      <limit lower="${-170 * pi / 180}" upper="${170 * pi / 180}"
+             effort="${max_effort}" velocity="${140 * pi / 180}" />
+      <safety_controller soft_lower_limit="${-168 * pi / 180}"
+                         soft_upper_limit="${168 * pi / 180}"
                          k_position="${safety_controller_k_pos}"
                          k_velocity="${safety_controller_k_vel}"/>
@@ -198,8 +197,8 @@
       <origin xyz="0 0 0" rpy="0 0 0"/>
       <axis xyz="0 1 0"/>
-      <limit lower="${-120 * PI / 180}" upper="${120 * PI / 180}"
-             effort="${max_effort}" velocity="${180 * PI / 180}" />
-      <safety_controller soft_lower_limit="${-118 * PI / 180}"
-                         soft_upper_limit="${118 * PI / 180}"
+      <limit lower="${-120 * pi / 180}" upper="${120 * pi / 180}"
+             effort="${max_effort}" velocity="${180 * pi / 180}" />
+      <safety_controller soft_lower_limit="${-118 * pi / 180}"
+                         soft_upper_limit="${118 * pi / 180}"
                          k_position="${safety_controller_k_pos}"
                          k_velocity="${safety_controller_k_vel}"/>
@@ -228,8 +227,8 @@
       <origin xyz="0 0 0" rpy="0 0 0"/>
       <axis xyz="0 0 1"/>
-      <limit lower="${-175 * PI / 180}" upper="${175 * PI / 180}"
-             effort="${max_effort}" velocity="${180 * PI / 180}" />
-      <safety_controller soft_lower_limit="${-173 * PI / 180}"
-                         soft_upper_limit="${173 * PI / 180}"
+      <limit lower="${-175 * pi / 180}" upper="${175 * pi / 180}"
+             effort="${max_effort}" velocity="${180 * pi / 180}" />
+      <safety_controller soft_lower_limit="${-173 * pi / 180}"
+                         soft_upper_limit="${173 * pi / 180}"
                          k_position="${safety_controller_k_pos}"
                          k_velocity="${safety_controller_k_vel}"/>

File: rll_description/urdf/rll_main.urdf.xacro (robot description, xacro)
@@ -4,10 +4,23 @@
   <xacro:include filename="$(find rll_description)/urdf/egl90/egl90_macro.xacro"/>
   <xacro:include filename="$(find rll_description)/urdf/visard160/rc_visard_160.xacro"/>
+  <xacro:include filename="$(find rll_description)/urdf/rll.gazebo.xacro"/>
+  <xacro:include filename="$(find rll_description)/urdf/rll.transmission.xacro"/>
   <!--  Arguments for the iiwa7 macro  -->
   <xacro:arg name="hardware_interface" default="PositionJointInterface"/>
   <xacro:arg name="robot_name" default="iiwa"/>
-  <link name="world">
+  <link name="world"/>
+  <joint name="table_joint" type="fixed">
+    <parent link="world" />
+    <child link="table" />
+    <origin xyz="0 0 0" rpy="0 0 0"/>
+  </joint>
+  <link name="table">
+    <inertial>
+      <origin xyz="0 0 0" rpy="0 0 0"/>
+      <mass value="0.1"/>
+      <inertia ixx="0.0001" ixy="0" ixz="0" iyy="0.0002" iyz="0" izz="0.0001"/>
+    </inertial>
     <visual>
-      <origin xyz="0 0 0" rpy="0 0 ${90 * PI / 180}"/>
+      <origin xyz="0 0 0" rpy="0 0 ${90 * pi / 180}"/>
       <geometry>
         <mesh filename="package://rll_description/meshes/rll/visual/table.dae"/>
@@ -114,5 +127,5 @@
       <origin xyz="0 0 0" rpy="0 0 0"/>
       <geometry>
-          <mesh filename="package://rll_description/meshes/rll/visual/base_adapter.dae"/>
+        <mesh filename="package://rll_description/meshes/rll/visual/base_adapter.dae"/>
       </geometry>
     </visual>
@@ -142,25 +155,4 @@
   </joint>
   <link name="$(arg robot_name)_gripper_link_ee"/>
-  <!-- gripper transmissions -->
-  <transmission name="$(arg robot_name)_tran_8">
-    <type>transmission_interface/SimpleTransmission</type>
-    <joint name="egl_position">
-      <hardwareInterface>hardware_interface/EffortJointInterface</hardwareInterface>
-    </joint>
-    <actuator name="$(arg robot_name)_motor_8">
-      <hardwareInterface>hardware_interface/EffortJointInterface</hardwareInterface>
-      <mechanicalReduction>1</mechanicalReduction>
-    </actuator>
-  </transmission>
-  <transmission name="$(arg robot_name)_tran_9">
-    <type>transmission_interface/SimpleTransmission</type>
-    <joint name="egl_position_mimic">
-      <hardwareInterface>hardware_interface/EffortJointInterface</hardwareInterface>
-    </joint>
-    <actuator name="$(arg robot_name)_motor_9">
-      <hardwareInterface>hardware_interface/EffortJointInterface</hardwareInterface>
-      <mechanicalReduction>1</mechanicalReduction>
-    </actuator>
-  </transmission>
   <joint name="profile_cams_joint" type="fixed">
     <parent link="world" />
@@ -170,5 +162,5 @@
   <link name="profile_cams">
     <visual>
-      <origin xyz="0 0 0" rpy="0 0 ${90 * PI / 180}"/>
+      <origin xyz="0 0 0" rpy="0 0 ${90 * pi / 180}"/>
       <geometry>
         <mesh filename="package://rll_description/meshes/rll/visual/profile_cams.dae"/>
@@ -184,14 +176,11 @@
   <!-- Roboception camera -->
   <xacro:rc_160 parent="profile_cams" prefix="$(arg robot_name)_">
-    <origin xyz="0.577 0.8 0.825" rpy="0 ${180 * PI / 180} 0"/>
+    <origin xyz="0.577 0.8 0.825" rpy="0 ${180 * pi / 180} 0"/>
   </xacro:rc_160>
-  <gazebo reference="world">
-    <static>true</static>
-  </gazebo>
-  <gazebo reference="$(arg robot_name)_base_adapter">
-    <static>true</static>
-  </gazebo>
   <material name="transparent">
     <color rgba="0.8784 0.8745 0.8588 0.3"/>
   </material>
+  <!--Extensions -->
+  <xacro:rll_gazebo robot_name="$(arg robot_name)" />
+  <xacro:rll_transmission hardware_interface="$(arg hardware_interface)" robot_name="$(arg robot_name)"/>
 </robot>

File: rll_description/urdf/visard160/rc_visard_160.xacro (robot description, xacro)
@@ -24,5 +24,5 @@
       <parent link="${prefix}roboception_gusset" />
       <child link="${prefix}roboception_adapter" />
-      <origin xyz="0.03 -0.075 0" rpy="${-90 * PI / 180} 0 ${135 * PI / 180}"/>
+      <origin xyz="0.03 -0.075 0" rpy="${-90 * pi / 180} 0 ${135 * pi / 180}"/>
     </joint>
     <link name="${prefix}roboception_adapter">
@@ -37,5 +37,5 @@
       <parent link="${prefix}roboception_adapter"/>
       <child link="${prefix}roboception_camera"/>
-      <origin xyz="-0.03 0.03 -0.08" rpy="${45 * PI / 180} ${-90 * PI / 180} 0"/>
+      <origin xyz="-0.03 0.03 -0.08" rpy="${45 * pi / 180} ${-90 * pi / 180} 0"/>
     </joint>
     <link name="${prefix}roboception_camera">

Commit message: gripper fixes and enforce joint limits from urdf
Signed-off-by: Wolfgang Wiedmeyer <wolfgang.wiedmeyer@kit.edu>

File: rll_description/urdf/egl90/egl90_macro.xacro (robot description, xacro)
@@ -38,4 +38,7 @@
           <mesh filename="package://rll_description/meshes/egl90/visual/gripper_base.stl" scale="0.001 0.001 0.001"/>
         </geometry>
+        <material name="black ">
+          <color rgba="1.0 1.0 1.0 1.0"/>
+        </material>
       </visual>
       <collision>
@@ -52,5 +55,5 @@
       <child link="${prefix}gripper_finger_right"/>
       <origin xyz="-0.013 0.1063 -0.1" rpy="0 ${180 * pi / 180} 0"/>
-      <axis xyz="1 0 0"/>
+      <axis xyz="0 0 1"/>
       <limit effort="100.0" lower="${min}" upper="${max}" velocity="100.0"/>
     </joint>
@@ -78,5 +81,5 @@
       <child link="${prefix}gripper_finger_left"/>
       <origin xyz="0.013 0.1063 -0.02" rpy="0 0 0"/>
-      <axis xyz="1 0 0"/>
+      <axis xyz="0 0 1"/>
       <limit effort="100.0" lower="${min}" upper="${max}" velocity="100.0"/>
     </joint>

File: rll_description/urdf/rll_main.urdf.xacro (robot description, xacro)
@@ -65,5 +65,5 @@
     <origin xyz="0 0 0.024" rpy="0 0 0"/>
   </xacro:egl90>
-  <xacro:egl90-jaws prefix="$(arg robot_name)_" min="-0.015" max="0.026">
+  <xacro:egl90-jaws prefix="$(arg robot_name)_" min="0" max="0.06">
     <mesh filename="package://rll_description/meshes/egl90/visual/gripper_finger.dae" scale="0.001 0.001 0.001"/>
   </xacro:egl90-jaws>

Commit message: description: various fixes, mainly for the base of the Axis camera
Thanks to Michael Mende for providing the Axis cam model!

Signed-off-by: Wolfgang Wiedmeyer <wolfgang.wiedmeyer@kit.edu>

File: rll_description/urdf/egl90/egl90_macro.xacro (robot description, xacro)
@@ -22,5 +22,5 @@
       </collision>
     </link>
-    <joint name="${prefix}mount" type="fixed">
+    <joint name="${prefix}gripper_mount" type="fixed">
       <parent link="${prefix}gripper_adapter"/>
       <child link="${prefix}gripper_base"/>

File: rll_description/urdf/rll_main.urdf.xacro (robot description, xacro)
@@ -107,5 +107,5 @@
     <parent link="profile_cams" />
     <child link="axis_cam_base" />
-    <origin xyz="0.577 0.8 1.13" rpy="${90 * pi / 180} 0 0"/>
+    <origin xyz="0.577 0.8 1.137" rpy="${90 * pi / 180} 0 0"/>
   </joint>
   <link name="axis_cam_base">

File: rll_description/urdf/visard160/rc_visard_160.xacro (robot description, xacro)
@@ -11,5 +11,5 @@
         <origin xyz="0 0 0" rpy="0 0 0"/>
         <geometry>
-          <mesh filename="package://rll_description/meshes/rll/visual/roboception_gusset.dae"/>
+          <mesh filename="package://rll_description/meshes/visard160/visual/roboception_gusset.dae"/>
         </geometry>
       </visual>
@@ -30,5 +30,5 @@
         <origin xyz="0 0 0" rpy="0 0 0"/>
         <geometry>
-          <mesh filename="package://rll_description/meshes/rll/visual/roboception_adapter.dae"/>
+          <mesh filename="package://rll_description/meshes/visard160/visual/roboception_adapter.dae"/>
         </geometry>
       </visual>

Commit message: Also add the robot prefix to the gripper joints
We need this for controlling several robots.

Signed-off-by: Wolfgang Wiedmeyer <wolfgang.wiedmeyer@kit.edu>

File: rll_description/urdf/egl90/egl90_macro.xacro (robot description, xacro)
@@ -51,5 +51,5 @@
   </xacro:macro>
   <xacro:macro name="egl90-jaws" params="prefix min max *mesh">
-    <joint name="egl_position" type="prismatic">
+    <joint name="${prefix}egl_position" type="prismatic">
       <parent link="${prefix}gripper_base"/>
       <child link="${prefix}gripper_finger_right"/>
@@ -77,5 +77,5 @@
       </collision>
     </link>
-    <joint name="egl_position_mimic" type="prismatic">
+    <joint name="${prefix}egl_position_mimic" type="prismatic">
       <parent link="${prefix}gripper_base"/>
       <child link="${prefix}gripper_finger_left"/>

File: rll_description/urdf/rll.transmission.xacro (robot description, xacro)
@@ -5,5 +5,5 @@
   <transmission name="$(arg robot_name)_tran_8">
     <type>transmission_interface/SimpleTransmission</type>
-    <joint name="egl_position">
+    <joint name="$(arg robot_name)_egl_position">
       <hardwareInterface>hardware_interface/EffortJointInterface</hardwareInterface>
     </joint>
@@ -16,5 +16,5 @@
   <transmission name="$(arg robot_name)_tran_9">
     <type>transmission_interface/SimpleTransmission</type>
-    <joint name="egl_position_mimic">
+    <joint name="$(arg robot_name)_egl_position_mimic">
       <hardwareInterface>hardware_interface/EffortJointInterface</hardwareInterface>
     </joint>
