Commit message: vastly improved gripper model and gripper control
Thanks to Michael Mende for creating the gripper model!

Signed-off-by: Wolfgang Wiedmeyer <wolfgang.wiedmeyer@kit.edu>

File: rll_description/urdf/egl90/egl90_macro.xacro (robot description, xacro)
@@ -1,20 +1,24 @@
 <?xml version="1.0"?>
 <robot name="egl90" xmlns:xacro="http://www.ros.org/wiki/xacro">
+  <xacro:property name="finger_visual_mesh_path" value="package://rll_description/meshes/egl90/visual/gripper_finger.dae" />
+  <xacro:property name="finger_collision_mesh_path" value="package://rll_description/meshes/egl90/collision/gripper_finger.stl" />
   <xacro:property name="finger_mass" value="0.1" />
-  <xacro:macro name="egl90" params="parent prefix *origin">
+  <xacro:property name="joint_lower_limit" value="0.0" />
+  <xacro:property name="joint_upper_limit" value="0.055" />
+  <xacro:macro name="egl90" params="parent prefix">
     <joint name="gripper_adapter_joint" type="fixed">
       <parent link="${parent}" />
       <child link="${prefix}gripper_adapter" />
-      <xacro:insert_block name="origin"/>
+      <origin xyz="0 0 0" rpy="0 0 ${-90 * pi / 180}"/>
     </joint>
     <link name="${prefix}gripper_adapter">
       <visual>
-        <origin xyz="0 0 0" rpy="${180 * pi / 180} 0 ${-90 * pi / 180}"/>
+        <origin xyz="0 0 0" rpy="0 0 0"/>
         <geometry>
-          <mesh filename="package://rll_description/meshes/egl90/visual/gripper_adapter.dae" scale="0.001 0.001 0.001"/>
+          <mesh filename="package://rll_description/meshes/egl90/visual/gripper_adapter.dae" />
         </geometry>
       </visual>
       <collision>
-        <origin xyz="0 0 -0.015" rpy="${180 * pi / 180} 0 ${-90 * pi / 180}"/>
+        <origin xyz="0 0 0.015" rpy="0 0 0"/>
         <geometry>
           <box size="0.09 0.07 0.03"/>
@@ -25,9 +29,9 @@
       <parent link="${prefix}gripper_adapter"/>
       <child link="${prefix}gripper_base"/>
-      <origin xyz="0 0.055 0" rpy="${90 * pi / 180} 0 ${180 * pi / 180}"/>
+      <origin xyz="0 0 0.024" rpy="0 0 0"/>
     </joint>
     <link name="${prefix}gripper_base">
       <inertial>
-        <origin xyz="0.055 0 0" rpy="${90 * pi / 180} 0 ${90 * pi / 180}"/>
+        <origin xyz="0 0 0" rpy="0 0 0"/>
         <mass value="0.3"/>
         <inertia ixx="0.0001" ixy="0" ixz="0" iyy="0.0002" iyz="0" izz="0.0001"/>
@@ -36,25 +40,84 @@
         <origin xyz="0 0 0" rpy="0 0 0" />
         <geometry>
-          <mesh filename="package://rll_description/meshes/egl90/visual/gripper_base.stl" scale="0.001 0.001 0.001"/>
+          <mesh filename="package://rll_description/meshes/egl90/visual/gripper_base.dae" />
         </geometry>
-        <material name="black ">
-          <color rgba="1.0 1.0 1.0 1.0"/>
-        </material>
       </visual>
       <collision>
-        <origin xyz="0 0.055 -0.025" rpy="0 0 0"/>
+        <origin xyz="-0.025 0 0.055" rpy="0 0 0"/>
         <geometry>
-          <box size="0.09 0.108 0.18"/>
+          <box size="0.18 0.09 0.108"/>
         </geometry>
       </collision>
     </link>
-  </xacro:macro>
-  <xacro:macro name="egl90-jaws" params="prefix min max *mesh">
-    <joint name="${prefix}egl_position" type="prismatic">
+    <joint name="${prefix}egl_position_left" type="prismatic">
       <parent link="${prefix}gripper_base"/>
+      <child link="${prefix}gripper_waggon_left"/>
+      <origin xyz="0.02985 0.0255 0.1063" rpy="0 0 ${180 * pi / 180}"/>
+      <axis xyz="1 0 0"/>
+      <limit effort="100.0" lower="${joint_lower_limit}" upper="${joint_upper_limit}" velocity="100.0"/>
+    </joint>
+    <link name="${prefix}gripper_waggon_left">
+      <visual>
+        <origin xyz="0 0 0" rpy="0 0 0"/>
+        <geometry>
+          <mesh filename="package://rll_description/meshes/egl90/visual/gripper_waggon.dae" />
+        </geometry>
+      </visual>
+      <collision>
+        <origin xyz="0 0 -0.01" rpy="0 0 0"/>
+        <geometry>
+          <box size="0.06 0.035 0.02"/>
+        </geometry>
+      </collision>
+    </link>
+    <joint name="${prefix}gripper_finger_left_joint" type="fixed">
+      <parent link="${prefix}gripper_waggon_left"/>
+      <child link="${prefix}gripper_finger_left"/>
+      <origin xyz="-0.016 0 0" rpy="0 0 0"/>
+    </joint>
+    <link name="${prefix}gripper_finger_left">
+      <inertial>
+        <origin xyz="0 0 0" rpy="0 0 0"/>
+        <mass value="${finger_mass}"/>
+        <inertia ixx="0.002" ixy="0" ixz="0" iyy="0.0002" iyz="0" izz="0.0002"/>
+      </inertial>
+      <visual>
+        <origin xyz="0 0 0" rpy="0 0 0"/>
+        <geometry>
+          <mesh filename="${finger_visual_mesh_path}" />
+        </geometry>
+      </visual>
+      <collision>
+        <origin xyz="0 0 0" rpy="0 0 0"/>
+        <geometry>
+          <mesh filename="${finger_collision_mesh_path}" />
+        </geometry>
+      </collision>
+    </link>
+    <joint name="${prefix}egl_position_right" type="prismatic">
+      <parent link="${prefix}gripper_base"/>
+      <child link="${prefix}gripper_waggon_right"/>
+      <origin xyz="-0.02985 -0.0255 0.1063" rpy="0 0 0"/>
+      <axis xyz="1 0 0"/>
+      <limit effort="100.0" lower="${joint_lower_limit}" upper="${joint_upper_limit}" velocity="100.0"/>
+    </joint>
+    <link name="${prefix}gripper_waggon_right">
+      <visual>
+        <origin xyz="0 0 0" rpy="0 0 0"/>
+        <geometry>
+          <mesh filename="package://rll_description/meshes/egl90/visual/gripper_waggon.dae" />
+        </geometry>
+      </visual>
+      <collision>
+        <origin xyz="0 0 -0.01" rpy="0 0 0"/>
+        <geometry>
+          <box size="0.06 0.035 0.02"/>
+        </geometry>
+      </collision>
+    </link>
+    <joint name="${prefix}gripper_finger_right_joint" type="fixed">
+      <parent link="${prefix}gripper_waggon_right"/>
       <child link="${prefix}gripper_finger_right"/>
-      <origin xyz="-0.013 0.1063 -0.1" rpy="0 ${180 * pi / 180} 0"/>
-      <axis xyz="0 0 1"/>
-      <limit effort="100.0" lower="${min}" upper="${max}" velocity="100.0"/>
+      <origin xyz="-0.016 0 0" rpy="0 0 0"/>
     </joint>
     <link name="${prefix}gripper_finger_right">
@@ -67,5 +130,5 @@
         <origin xyz="0 0 0" rpy="0 0 0"/>
         <geometry>
-          <xacro:insert_block name="mesh"/>
+          <mesh filename="${finger_visual_mesh_path}" />
         </geometry>
       </visual>
@@ -73,31 +136,5 @@
         <origin xyz="0 0 0" rpy="0 0 0"/>
         <geometry>
-          <xacro:insert_block name="mesh"/>
-        </geometry>
-      </collision>
-    </link>
-    <joint name="${prefix}egl_position_mimic" type="prismatic">
-      <parent link="${prefix}gripper_base"/>
-      <child link="${prefix}gripper_finger_left"/>
-      <origin xyz="0.013 0.1063 -0.02" rpy="0 0 0"/>
-      <axis xyz="0 0 1"/>
-      <limit effort="100.0" lower="${min}" upper="${max}" velocity="100.0"/>
-    </joint>
-    <link name="${prefix}gripper_finger_left">
-      <inertial>
-        <origin xyz="0 0 0" rpy="0 0 0"/>
-        <mass value="${finger_mass}"/>
-        <inertia ixx="0.002" ixy="0" ixz="0" iyy="0.0002" iyz="0" izz="0.0002"/>
-      </inertial>
-      <visual>
-        <origin xyz="0 0 0" rpy="0 0 0"/>
-        <geometry>
-          <xacro:insert_block name="mesh"/>
-        </geometry>
-      </visual>
-      <collision>
-        <origin xyz="0 0 0" rpy="0 0 0"/>
-        <geometry>
-          <xacro:insert_block name="mesh"/>
+          <mesh filename="${finger_collision_mesh_path}" />
         </geometry>
       </collision>

File: rll_description/urdf/rll.transmission.xacro (robot description, xacro)
@@ -2,26 +2,26 @@
 <robot xmlns:xacro="http://www.ros.org/wiki/xacro">
   <xacro:macro name="rll_transmission" params="hardware_interface robot_name">
-   <!-- gripper right transmissions -->
-  <transmission name="$(arg robot_name)_tran_8">
-    <type>transmission_interface/SimpleTransmission</type>
-    <joint name="$(arg robot_name)_egl_position">
-      <hardwareInterface>hardware_interface/EffortJointInterface</hardwareInterface>
-    </joint>
-    <actuator name="$(arg robot_name)_motor_8">
-      <hardwareInterface>hardware_interface/EffortJointInterface</hardwareInterface>
+    <!-- gripper right transmissions -->
+    <transmission name="$(arg robot_name)_tran_8">
+      <type>transmission_interface/SimpleTransmission</type>
+      <joint name="$(arg robot_name)_egl_position_left">
+        <hardwareInterface>hardware_interface/EffortJointInterface</hardwareInterface>
+      </joint>
+      <actuator name="$(arg robot_name)_motor_8">
+        <hardwareInterface>hardware_interface/EffortJointInterface</hardwareInterface>
+        <mechanicalReduction>1</mechanicalReduction>
+      </actuator>
+    </transmission>
+    <!-- gripper left transmissions -->
+    <transmission name="$(arg robot_name)_tran_9">
+      <type>transmission_interface/SimpleTransmission</type>
+      <joint name="$(arg robot_name)_egl_position_right">
+        <hardwareInterface>hardware_interface/EffortJointInterface</hardwareInterface>
+      </joint>
+      <actuator name="$(arg robot_name)_motor_9">
+        <hardwareInterface>hardware_interface/EffortJointInterface</hardwareInterface>
       <mechanicalReduction>1</mechanicalReduction>
     </actuator>
-  </transmission>
-   <!-- gripper left transmissions -->
-  <transmission name="$(arg robot_name)_tran_9">
-    <type>transmission_interface/SimpleTransmission</type>
-    <joint name="$(arg robot_name)_egl_position_mimic">
-      <hardwareInterface>hardware_interface/EffortJointInterface</hardwareInterface>
-    </joint>
-    <actuator name="$(arg robot_name)_motor_9">
-      <hardwareInterface>hardware_interface/EffortJointInterface</hardwareInterface>
-      <mechanicalReduction>1</mechanicalReduction>
-    </actuator>
-  </transmission>
-  </xacro:macro>
-</robot>
+    </transmission>
+    </xacro:macro>
+  </robot>

File: rll_description/urdf/rll_main.urdf.xacro (robot description, xacro)
@@ -62,10 +62,5 @@
   </xacro:iiwa7>
   <!-- Here we insert a Schunk gripper in the scene -->
-  <xacro:egl90 parent="$(arg robot_name)_link_ee" prefix="$(arg robot_name)_">
-    <origin xyz="0 0 0.024" rpy="0 0 0"/>
-  </xacro:egl90>
-  <xacro:egl90-jaws prefix="$(arg robot_name)_" min="0" max="0.06">
-    <mesh filename="package://rll_description/meshes/egl90/visual/gripper_finger.dae" scale="0.001 0.001 0.001"/>
-  </xacro:egl90-jaws>
+  <xacro:egl90 parent="$(arg robot_name)_link_ee" prefix="$(arg robot_name)_" />
   <!-- TCP link -->
   <joint name="gripper_ee_joint" type="fixed">
@@ -119,5 +114,5 @@
       <origin xyz="0 0 0.035" rpy="0 0 0"/>
       <geometry>
-        <box size="0.01 0.01 0.07"/>
+        <box size="0.07 0.07 0.07"/>
       </geometry>
     </collision>

Commit message: a little parameter tuning for grasping in simulation
Signed-off-by: Wolfgang Wiedmeyer <wolfgang.wiedmeyer@kit.edu>

File: rll_description/urdf/egl90/egl90_macro.xacro (robot description, xacro)
@@ -55,5 +55,5 @@
       <origin xyz="0.02985 0.0255 0.1063" rpy="0 0 ${180 * pi / 180}"/>
       <axis xyz="1 0 0"/>
-      <limit effort="100.0" lower="${joint_lower_limit}" upper="${joint_upper_limit}" velocity="100.0"/>
+      <limit effort="1000.0" lower="${joint_lower_limit}" upper="${joint_upper_limit}" velocity="100.0"/>
     </joint>
     <link name="${prefix}gripper_waggon_left">
@@ -100,5 +100,5 @@
       <origin xyz="-0.02985 -0.0255 0.1063" rpy="0 0 0"/>
       <axis xyz="1 0 0"/>
-      <limit effort="100.0" lower="${joint_lower_limit}" upper="${joint_upper_limit}" velocity="100.0"/>
+      <limit effort="1000.0" lower="${joint_lower_limit}" upper="${joint_upper_limit}" velocity="100.0"/>
     </joint>
     <link name="${prefix}gripper_waggon_right">

File: rll_description/urdf/rll.gazebo.xacro (robot description, xacro)
@@ -4,7 +4,11 @@
     <!-- Link Table -->
     <gazebo reference="table">
-      <mu1>1.0</mu1>
-      <mu2>1.0</mu2>
-      <static>true</static>
+      <mu1>100.0</mu1>
+      <mu2>100.0</mu2>
+      <!-- <kp>1000000.0</kp> -->
+      <!-- <kd>1.0</kd> -->
+      <!-- <fdir1>0 0 1</fdir1> -->
+      <!-- <minDepth>0.001</minDepth> -->
+      <!-- <static>true</static> -->
     </gazebo>
     <gazebo reference="$(arg robot_name)_link_0">
@@ -14,8 +18,40 @@
       <mu1>1.0</mu1>
       <mu2>1.0</mu2>
+      <!-- <kp>1000000.0</kp> -->
+      <!-- <kd>1.0</kd> -->
+      <!-- <fdir1>1 0 0</fdir1> -->
+      <!-- <minDepth>0.002</minDepth> -->
+      <!-- <maxContacts>2</maxContacts> -->
+      <!-- <maxVel>0</maxVel> -->
     </gazebo>
     <gazebo reference="$(arg robot_name)_gripper_waggon_left">
       <mu1>1.0</mu1>
       <mu2>1.0</mu2>
+      <!-- <kp>1000000.0</kp> -->
+      <!-- <kd>1.0</kd> -->
+      <!-- <fdir1>1 0 0</fdir1> -->
+      <!-- <minDepth>0.002</minDepth> -->
+      <!-- <maxContacts>2</maxContacts> -->
+      <!-- <maxVel>0</maxVel> -->
+    </gazebo>
+    <gazebo reference="$(arg robot_name)_gripper_finger_right">
+      <mu1>1.0</mu1>
+      <mu2>1.0</mu2>
+      <!-- <kp>1000000.0</kp> -->
+      <!-- <kd>1.0</kd> -->
+      <!-- <fdir1>1 0 0</fdir1> -->
+      <!-- <minDepth>0.002</minDepth> -->
+      <!-- <maxContacts>2</maxContacts> -->
+      <!-- <maxVel>0</maxVel> -->
+    </gazebo>
+    <gazebo reference="$(arg robot_name)_gripper_finger_left">
+      <mu1>1.0</mu1>
+      <mu2>1.0</mu2>
+      <!-- <kp>1000000.0</kp> -->
+      <!-- <kd>1.0</kd> -->
+      <!-- <fdir1>1 0 0</fdir1> -->
+      <!-- <minDepth>0.002</minDepth> -->
+      <!-- <maxContacts>2</maxContacts> -->
+      <!-- <maxVel>0</maxVel> -->
     </gazebo>
     <!-- Link profile_cams -->
@@ -33,5 +69,5 @@
         </arm>
         <forces_angle_tolerance>100</forces_angle_tolerance>
-        <update_rate>30</update_rate>
+        <update_rate>100</update_rate>
         <grip_count_threshold>4</grip_count_threshold>
         <max_grip_count>8</max_grip_count>

Commit message: updated moment of inertia for the table and the gripper

File: rll_description/urdf/egl90/egl90_macro.xacro (robot description, xacro)
@@ -33,7 +33,7 @@
     <link name="${prefix}gripper_base">
       <inertial>
-        <origin xyz="0 0 0" rpy="0 0 0"/>
-        <mass value="0.3"/>
-        <inertia ixx="0.0001" ixy="0" ixz="0" iyy="0.0002" iyz="0" izz="0.0001"/>
+        <origin xyz="0 0 0.0465291" rpy="0 0 0"/>
+        <mass value="1.8"/>
+        <inertia ixx="0.0024631" ixy="0" ixz="0" iyy="0.0032423" iyz="0" izz="0.0030708"/>
       </inertial>
       <visual>

File: rll_description/urdf/rll_cell.xacro (robot description, xacro)
@@ -19,7 +19,7 @@
     <link name="table">
       <inertial>
-        <origin xyz="0 0 0" rpy="0 0 0"/>
+        <origin xyz="0 0 -0.18746" rpy="0 0 0"/>
         <mass value="600"/>
-        <inertia ixx="1" ixy="0" ixz="0" iyy="1" iyz="0" izz="1"/>
+        <inertia ixx="152.284" ixy="0" ixz="0" iyy="207.558" iyz="0" izz="288.142"/>
       </inertial>
       <visual>

Commit message: gripper description: set more reasonable limit
Signed-off-by: Wolfgang Wiedmeyer <wolfgang.wiedmeyer@kit.edu>

File: rll_description/urdf/egl90/egl90_macro.xacro (robot description, xacro)
@@ -55,5 +55,5 @@
       <origin xyz="0.02985 0.0255 0.1063" rpy="0 0 ${180 * pi / 180}"/>
       <axis xyz="1 0 0"/>
-      <limit effort="1000.0" lower="${joint_lower_limit}" upper="${joint_upper_limit}" velocity="100.0"/>
+      <limit effort="500.0" lower="${joint_lower_limit}" upper="${joint_upper_limit}" velocity="2.0"/>
     </joint>
     <link name="${prefix}gripper_waggon_left">
@@ -100,5 +100,5 @@
       <origin xyz="-0.02985 -0.0255 0.1063" rpy="0 0 0"/>
       <axis xyz="1 0 0"/>
-      <limit effort="1000.0" lower="${joint_lower_limit}" upper="${joint_upper_limit}" velocity="100.0"/>
+      <limit effort="500.0" lower="${joint_lower_limit}" upper="${joint_upper_limit}" velocity="2.0"/>
     </joint>
     <link name="${prefix}gripper_waggon_right">

Commit message: desc: reduce max gripper velocity

File: rll_description/urdf/egl90/egl90_macro.xacro (robot description, xacro)
@@ -55,5 +55,5 @@
       <origin xyz="0.02985 0.0255 0.1063" rpy="0 0 ${180 * pi / 180}"/>
       <axis xyz="1 0 0"/>
-      <limit effort="500.0" lower="${joint_lower_limit}" upper="${joint_upper_limit}" velocity="2.0"/>
+      <limit effort="500.0" lower="${joint_lower_limit}" upper="${joint_upper_limit}" velocity="0.1"/>
     </joint>
     <link name="${prefix}gripper_waggon_left">
@@ -100,5 +100,5 @@
       <origin xyz="-0.02985 -0.0255 0.1063" rpy="0 0 0"/>
       <axis xyz="1 0 0"/>
-      <limit effort="500.0" lower="${joint_lower_limit}" upper="${joint_upper_limit}" velocity="2.0"/>
+      <limit effort="500.0" lower="${joint_lower_limit}" upper="${joint_upper_limit}" velocity="0.1"/>
     </joint>
     <link name="${prefix}gripper_waggon_right">
