Commit message: description: various fixes for dynamics properties and controller settings
The inertia parameters for the EGL gripper are updated with the values
from the identification by the Sunrise controller. The real joint torque
limits are added for the iiwa7. The table inertias are set to more
realistic values.

The legacy mode tag is not needed anymore for the Gazebo ROS control
interface. The Gazebo grasp fix plugin settings are updated to make it
attach grasp objects right away on first contact while keeping the update
rate low.
The iiwa actuator hardware interfaces need to be prepended with
"hardware_interface". The safety controller pos and vel factors are set to
more sensible values.

The surface property settings are cleaned up. Unless more fine-grained
settings are needed in the future, it is enough to set mu1 and mu2.

Signed-off-by: Wolfgang Wiedmeyer <wolfgang.wiedmeyer@kit.edu>

File: rll_description/urdf/egl90/egl90_macro.xacro (robot description, xacro)
@@ -34,6 +34,6 @@
       <inertial>
         <origin xyz="0 0 0.0465291" rpy="0 0 0"/>
-        <mass value="1.8"/>
-        <inertia ixx="0.0024631" ixy="0" ixz="0" iyy="0.0032423" iyz="0" izz="0.0030708"/>
+        <mass value="2.57"/>
+	<inertia ixx="0.003" ixy="0" ixz="0" iyy="0.004" iyz="0" izz="0.004"/>
       </inertial>
       <visual>

File: rll_description/urdf/iiwa7/iiwa.gazebo.xacro (robot description, xacro)
@@ -6,5 +6,4 @@
       <plugin name="gazebo_ros_control" filename="libgazebo_ros_control.so">
         <robotNamespace>/${robot_name}</robotNamespace>
-        <legacyModeNS>true</legacyModeNS>
       </plugin>
     </gazebo>

File: rll_description/urdf/iiwa7/iiwa.transmission.xacro (robot description, xacro)
@@ -9,5 +9,5 @@
       </joint>
       <actuator name="${robot_name}_motor_1">
-	<hardwareInterface>${hardware_interface}</hardwareInterface>
+	<hardwareInterface>hardware_interface/${hardware_interface}</hardwareInterface>
 	<mechanicalReduction>1</mechanicalReduction>
       </actuator>
@@ -20,5 +20,5 @@
       </joint>
       <actuator name="${robot_name}_motor_2">
-	<hardwareInterface>${hardware_interface}</hardwareInterface>
+	<hardwareInterface>hardware_interface/${hardware_interface}</hardwareInterface>
 	<mechanicalReduction>1</mechanicalReduction>
       </actuator>
@@ -31,5 +31,5 @@
       </joint>
       <actuator name="${robot_name}_motor_3">
-	<hardwareInterface>${hardware_interface}</hardwareInterface>
+	<hardwareInterface>hardware_interface/${hardware_interface}</hardwareInterface>
 	<mechanicalReduction>1</mechanicalReduction>
       </actuator>
@@ -42,5 +42,5 @@
       </joint>
       <actuator name="${robot_name}_motor_4">
-	<hardwareInterface>${hardware_interface}</hardwareInterface>
+	<hardwareInterface>hardware_interface/${hardware_interface}</hardwareInterface>
 	<mechanicalReduction>1</mechanicalReduction>
       </actuator>
@@ -53,5 +53,5 @@
       </joint>
       <actuator name="${robot_name}_motor_5">
-	<hardwareInterface>${hardware_interface}</hardwareInterface>
+	<hardwareInterface>hardware_interface/${hardware_interface}</hardwareInterface>
 	<mechanicalReduction>1</mechanicalReduction>
       </actuator>
@@ -64,5 +64,5 @@
       </joint>
       <actuator name="${robot_name}_motor_6">
-	<hardwareInterface>${hardware_interface}</hardwareInterface>
+	<hardwareInterface>hardware_interface/${hardware_interface}</hardwareInterface>
 	<mechanicalReduction>1</mechanicalReduction>
       </actuator>
@@ -75,5 +75,5 @@
       </joint>
       <actuator name="${robot_name}_motor_7">
-	<hardwareInterface>${hardware_interface}</hardwareInterface>
+	<hardwareInterface>hardware_interface/${hardware_interface}</hardwareInterface>
 	<mechanicalReduction>1</mechanicalReduction>
       </actuator>

File: rll_description/urdf/iiwa7/iiwa7.xacro (robot description, xacro)
@@ -5,10 +5,7 @@
   <!-- Import Transmissions -->
   <xacro:include filename="$(find rll_description)/urdf/iiwa7/iiwa.transmission.xacro" />
-  <!-- some constants -->
-  <xacro:property name="safety_controller_k_pos" value="100" />
-  <xacro:property name="safety_controller_k_vel" value="2" />
+  <xacro:property name="safety_controller_k_pos" value="15" />
+  <xacro:property name="safety_controller_k_vel" value="10" />
   <xacro:property name="joint_damping" value="0.5" />
-  <!-- TODO: set the correct individual effort values for every joint -->
-  <xacro:property name="max_effort" value="300"/>
   <xacro:macro name="iiwa7" params="parent hardware_interface robot_name *origin">
     <!--joint between {parent} and link_0-->
@@ -48,5 +45,5 @@
       <axis xyz="0 0 1"/>
       <limit lower="${-169 * pi / 180}" upper="${169 * pi / 180}"
-             effort="${max_effort}" velocity="${98 * pi / 180}" />
+             effort="176" velocity="${98 * pi / 180}" />
       <safety_controller soft_lower_limit="${-167 * pi / 180}"
                          soft_upper_limit="${167 * pi / 180}"
@@ -78,5 +75,5 @@
       <axis xyz="0 1 0"/>
       <limit lower="${-119 * pi / 180}" upper="${119 * pi / 180}"
-             effort="${max_effort}" velocity="${98 * pi / 180}" />
+             effort="176" velocity="${98 * pi / 180}" />
       <safety_controller soft_lower_limit="${-117 * pi / 180}"
                          soft_upper_limit="${117 * pi / 180}"
@@ -108,5 +105,5 @@
       <axis xyz="0 0 1"/>
       <limit lower="${-169 * pi / 180}" upper="${169 * pi / 180}"
-             effort="${max_effort}" velocity="${100 * pi / 180}" />
+             effort="110" velocity="${100 * pi / 180}" />
       <safety_controller soft_lower_limit="${-167 * pi / 180}"
                          soft_upper_limit="${167 * pi / 180}"
@@ -138,5 +135,5 @@
       <axis xyz="0 -1 0"/>
       <limit lower="${-119 * pi / 180}" upper="${119 * pi / 180}"
-             effort="${max_effort}" velocity="${130 * pi / 180}" />
+             effort="110" velocity="${130 * pi / 180}" />
       <safety_controller soft_lower_limit="${-117 * pi / 180}"
                          soft_upper_limit="${117 * pi / 180}"
@@ -168,5 +165,5 @@
       <axis xyz="0 0 1"/>
       <limit lower="${-169 * pi / 180}" upper="${169 * pi / 180}"
-             effort="${max_effort}" velocity="${140 * pi / 180}" />
+             effort="110" velocity="${140 * pi / 180}" />
       <safety_controller soft_lower_limit="${-167 * pi / 180}"
                          soft_upper_limit="${167 * pi / 180}"
@@ -198,5 +195,5 @@
       <axis xyz="0 1 0"/>
       <limit lower="${-119 * pi / 180}" upper="${119 * pi / 180}"
-             effort="${max_effort}" velocity="${180 * pi / 180}" />
+             effort="40" velocity="${180 * pi / 180}" />
       <safety_controller soft_lower_limit="${-117 * pi / 180}"
                          soft_upper_limit="${117 * pi / 180}"
@@ -228,5 +225,5 @@
       <axis xyz="0 0 1"/>
       <limit lower="${-174 * pi / 180}" upper="${174 * pi / 180}"
-             effort="${max_effort}" velocity="${180 * pi / 180}" />
+             effort="40" velocity="${180 * pi / 180}" />
       <safety_controller soft_lower_limit="${-172 * pi / 180}"
                          soft_upper_limit="${172 * pi / 180}"
@@ -238,5 +235,5 @@
       <inertial>
         <origin xyz="0 0 0.1" rpy="0 0 0"/>
-        <mass value="3.129"/>
+        <mass value="0.34217"/>
         <inertia ixx="0.0022711"  ixy="0.0000221"  ixz="0" iyy="0.0022807" iyz="0" izz="0.002872" />
       </inertial>

File: rll_description/urdf/rll.gazebo.xacro (robot description, xacro)
@@ -4,58 +4,14 @@
     <!-- Link Table -->
     <gazebo reference="table">
-      <mu1>100.0</mu1>
-      <mu2>100.0</mu2>
-      <kp>1000000.0</kp>
-      <kd>1.0</kd>
-      <fdir1>1 0 0</fdir1>
-      <minDepth>0.001</minDepth>
-      <!-- <static>true</static> -->
-    </gazebo>
-    <gazebo reference="$(arg robot_name)_link_0">
-      <static>true</static>
+      <mu1>10.0</mu1>
+      <mu2>10.0</mu2>
     </gazebo>
     <gazebo reference="$(arg robot_name)_gripper_waggon_right">
-      <mu1>1.0</mu1>
-      <mu2>1.0</mu2>
-      <!-- <kp>1000000.0</kp> -->
-      <!-- <kd>1.0</kd> -->
-      <!-- <fdir1>1 0 0</fdir1> -->
-      <!-- <minDepth>0.002</minDepth> -->
-      <!-- <maxContacts>2</maxContacts> -->
-      <!-- <maxVel>0</maxVel> -->
+      <mu1>10.0</mu1>
+      <mu2>10.0</mu2>
     </gazebo>
     <gazebo reference="$(arg robot_name)_gripper_waggon_left">
-      <mu1>1.0</mu1>
-      <mu2>1.0</mu2>
-      <!-- <kp>1000000.0</kp> -->
-      <!-- <kd>1.0</kd> -->
-      <!-- <fdir1>1 0 0</fdir1> -->
-      <!-- <minDepth>0.002</minDepth> -->
-      <!-- <maxContacts>2</maxContacts> -->
-      <!-- <maxVel>0</maxVel> -->
-    </gazebo>
-    <gazebo reference="$(arg robot_name)_gripper_finger_right">
-      <mu1>1.0</mu1>
-      <mu2>1.0</mu2>
-      <!-- <kp>1000000.0</kp> -->
-      <!-- <kd>1.0</kd> -->
-      <!-- <fdir1>1 0 0</fdir1> -->
-      <!-- <minDepth>0.002</minDepth> -->
-      <!-- <maxContacts>2</maxContacts> -->
-      <!-- <maxVel>0</maxVel> -->
-    </gazebo>
-    <gazebo reference="$(arg robot_name)_gripper_finger_left">
-      <mu1>1.0</mu1>
-      <mu2>1.0</mu2>
-      <!-- <kp>1000000.0</kp> -->
-      <!-- <kd>1.0</kd> -->
-      <!-- <fdir1>1 0 0</fdir1> -->
-      <!-- <minDepth>0.002</minDepth> -->
-      <!-- <maxContacts>2</maxContacts> -->
-      <!-- <maxVel>0</maxVel> -->
-    </gazebo>
-    <!-- Link profile_cams -->
-    <gazebo reference="profile_cams">
-      <static>true</static>
+      <mu1>10.0</mu1>
+      <mu2>10.0</mu2>
     </gazebo>
     <!-- grasp plugin -->
@@ -69,8 +25,8 @@
         </arm>
         <forces_angle_tolerance>100</forces_angle_tolerance>
-        <update_rate>100</update_rate>
-        <grip_count_threshold>4</grip_count_threshold>
-        <max_grip_count>8</max_grip_count>
-        <release_tolerance>0.0005</release_tolerance>
+        <update_rate>20</update_rate>
+        <grip_count_threshold>1</grip_count_threshold>
+        <max_grip_count>2</max_grip_count>
+        <release_tolerance>0.005</release_tolerance>
         <disable_collisions_on_attach>false</disable_collisions_on_attach>
         <contact_topic>__default_topic__</contact_topic>

File: rll_description/urdf/rll_cell.xacro (robot description, xacro)
@@ -19,7 +19,7 @@
     <link name="table">
       <inertial>
-        <origin xyz="0 0 -0.18746" rpy="0 0 0"/>
-        <mass value="600"/>
-        <inertia ixx="152.284" ixy="0" ixz="0" iyy="207.558" iyz="0" izz="288.142"/>
+        <origin xyz="0 0 -0.1" rpy="0 0 0"/>
+        <mass value="500"/>
+        <inertia ixx="108" ixy="0" ixz="0" iyy="62" iyz="0" izz="167"/>
       </inertial>
       <visual>
@@ -32,7 +32,4 @@
         <origin xyz="0 0 -0.1" rpy="0 0 0"/>
         <geometry>
-          <!-- for disallowing eef positions below joint 1 -->
-          <!-- <box size="1.2 1.6 0.49"/> -->
-          <!-- for grasping objects on table -->
           <box size="1.2 1.6 0.2"/>
         </geometry>
