Commit message: description: move egl90 Gazebo and transmission settings to egl90 folder
Settings for the gripper should be separated from general work cell settings.

Signed-off-by: Wolfgang Wiedmeyer <wolfgang.wiedmeyer@kit.edu>

File: rll_description/urdf/egl90/egl90.transmission.xacro (robot description, xacro)
@@ -1,12 +1,12 @@
 <?xml version="1.0"?>
 <robot xmlns:xacro="http://www.ros.org/wiki/xacro">
-  <xacro:macro name="rll_transmission" params="hardware_interface robot_name">
+  <xacro:macro name="egl90_transmission" params="robot_name">
     <!-- gripper right transmissions -->
-    <transmission name="$(arg robot_name)_tran_8">
+    <transmission name="$(arg robot_name)_tran_egl_position_left">
       <type>transmission_interface/SimpleTransmission</type>
       <joint name="$(arg robot_name)_egl_position_left">
         <hardwareInterface>hardware_interface/EffortJointInterface</hardwareInterface>
       </joint>
-      <actuator name="$(arg robot_name)_motor_8">
+      <actuator name="$(arg robot_name)_motor_egl_position_left">
         <hardwareInterface>hardware_interface/EffortJointInterface</hardwareInterface>
         <mechanicalReduction>1</mechanicalReduction>
@@ -14,10 +14,10 @@
     </transmission>
     <!-- gripper left transmissions -->
-    <transmission name="$(arg robot_name)_tran_9">
+    <transmission name="$(arg robot_name)_tran_egl_position_right">
       <type>transmission_interface/SimpleTransmission</type>
       <joint name="$(arg robot_name)_egl_position_right">
         <hardwareInterface>hardware_interface/EffortJointInterface</hardwareInterface>
       </joint>
-      <actuator name="$(arg robot_name)_motor_9">
+      <actuator name="$(arg robot_name)_motor_egl_position_right">
         <hardwareInterface>hardware_interface/EffortJointInterface</hardwareInterface>
       <mechanicalReduction>1</mechanicalReduction>

File: rll_description/urdf/egl90/egl90.xacro (robot description, xacro)
@@ -1,4 +1,6 @@
 <?xml version="1.0"?>
 <robot name="egl90" xmlns:xacro="http://www.ros.org/wiki/xacro">
+  <xacro:include filename="$(find rll_description)/urdf/egl90/egl90.gazebo.xacro" />
+  <xacro:include filename="$(find rll_description)/urdf/egl90/egl90.transmission.xacro" />
   <xacro:property name="finger_visual_mesh_path" value="package://rll_description/meshes/egl90/visual/gripper_finger.dae" />
   <xacro:property name="finger_collision_mesh_path" value="package://rll_description/meshes/egl90/collision/gripper_finger.stl" />
@@ -140,4 +142,13 @@
       </collision>
     </link>
+    <!-- TCP link -->
+    <joint name="gripper_ee_joint" type="fixed">
+      <parent link="$(arg robot_name)_link_ee" />
+      <child link="$(arg robot_name)_gripper_link_ee" />
+      <origin xyz="0 0 0.248" rpy="0 0 0"/>
+    </joint>
+    <link name="$(arg robot_name)_gripper_link_ee"/>
+    <xacro:egl90_gazebo robot_name="${robot_name}" />
+    <xacro:egl90_transmission robot_name="${robot_name}" />
   </xacro:macro>
 </robot>

File: rll_description/urdf/iiwa7/iiwa.transmission.xacro (robot description, xacro)
@@ -1,5 +1,5 @@
 <?xml version="1.0"?>
 <robot xmlns:xacro="http://www.ros.org/wiki/xacro">
-  <xacro:macro name="iiwa_transmission" params="hardware_interface">
+  <xacro:macro name="iiwa_transmission" params="robot_name hardware_interface">
     <transmission name="${robot_name}_tran_1">
       <robotNamespace>/${robot_name}</robotNamespace>

File: rll_description/urdf/iiwa7/iiwa7.xacro (robot description, xacro)
@@ -1,7 +1,5 @@
 <?xml version="1.0"?>
 <robot xmlns:xacro="http://www.ros.org/wiki/xacro">
-  <!-- Import all Gazebo-customization elements, including Gazebo colors -->
   <xacro:include filename="$(find rll_description)/urdf/iiwa7/iiwa.gazebo.xacro" />
-  <!-- Import Transmissions -->
   <xacro:include filename="$(find rll_description)/urdf/iiwa7/iiwa.transmission.xacro" />
   <xacro:property name="safety_controller_k_pos" value="15" />
@@ -256,7 +254,7 @@
     <link name="${robot_name}_link_ee">
     </link>
-    <!--Extensions -->
     <xacro:iiwa_gazebo robot_name="${robot_name}" />
-    <xacro:iiwa_transmission hardware_interface="${hardware_interface}"/>
+    <xacro:iiwa_transmission robot_name="${robot_name}"
+			     hardware_interface="${hardware_interface}"/>
   </xacro:macro>
 </robot>

File: rll_description/urdf/rll.gazebo.xacro (robot description, xacro)
@@ -7,30 +7,4 @@
       <mu2>10.0</mu2>
     </gazebo>
-    <gazebo reference="$(arg robot_name)_gripper_waggon_right">
-      <mu1>10.0</mu1>
-      <mu2>10.0</mu2>
-    </gazebo>
-    <gazebo reference="$(arg robot_name)_gripper_waggon_left">
-      <mu1>10.0</mu1>
-      <mu2>10.0</mu2>
-    </gazebo>
-    <!-- grasp plugin -->
-    <gazebo>
-      <plugin name="gazebo_grasp_fix" filename="libgazebo_grasp_fix.so">
-        <arm>
-          <arm_name>$(arg robot_name)</arm_name>
-          <palm_link>$(arg robot_name)_link_7</palm_link>
-          <gripper_link>$(arg robot_name)_gripper_waggon_right</gripper_link>
-          <gripper_link>$(arg robot_name)_gripper_waggon_left</gripper_link>
-        </arm>
-        <forces_angle_tolerance>100</forces_angle_tolerance>
-        <update_rate>20</update_rate>
-        <grip_count_threshold>1</grip_count_threshold>
-        <max_grip_count>2</max_grip_count>
-        <release_tolerance>0.005</release_tolerance>
-        <disable_collisions_on_attach>false</disable_collisions_on_attach>
-        <contact_topic>__default_topic__</contact_topic>
-      </plugin>
-    </gazebo>
   </xacro:macro>
 </robot>

File: rll_description/urdf/rll_cell.xacro (robot description, xacro)
@@ -2,9 +2,8 @@
 <robot xmlns:xacro="http://www.ros.org/wiki/xacro" name="rll_cell">
   <xacro:include filename="$(find rll_description)/urdf/iiwa7/iiwa7.xacro"/>
-  <xacro:include filename="$(find rll_description)/urdf/egl90/egl90_macro.xacro"/>
+  <xacro:include filename="$(find rll_description)/urdf/egl90/egl90.xacro"/>
   <xacro:include filename="$(find rll_description)/urdf/visard160/rc_visard_160.xacro"/>
   <xacro:include filename="$(find rll_description)/urdf/rll_virtual.xacro"/>
   <xacro:include filename="$(find rll_description)/urdf/rll.gazebo.xacro"/>
-  <xacro:include filename="$(find rll_description)/urdf/rll.transmission.xacro"/>
   <!--  Arguments for the iiwa7 macro  -->
   <xacro:arg name="hardware_interface" default="PositionJointInterface"/>
@@ -60,11 +59,4 @@
     <!-- Here we insert a Schunk gripper in the scene -->
     <xacro:egl90 parent="$(arg robot_name)_link_ee" prefix="$(arg robot_name)_" />
-    <!-- TCP link -->
-    <joint name="gripper_ee_joint" type="fixed">
-      <parent link="$(arg robot_name)_link_ee" />
-      <child link="$(arg robot_name)_gripper_link_ee" />
-      <origin xyz="0 0 0.248" rpy="0 0 0"/>
-    </joint>
-    <link name="$(arg robot_name)_gripper_link_ee"/>
     <joint name="profile_cams_joint" type="fixed">
       <parent link="world" />
@@ -137,5 +129,4 @@
     <xacro:rll_virtual />
     <xacro:rll_gazebo robot_name="$(arg robot_name)" />
-    <xacro:rll_transmission hardware_interface="$(arg hardware_interface)" robot_name="$(arg robot_name)"/>
 </xacro:macro>
 </robot>
