Commit message: description: set damping for the gripper joints
This seems to help with occasional oscillations of the gripper fingers
when grasping.

Signed-off-by: Wolfgang Wiedmeyer <wolfgang.wiedmeyer@kit.edu>

File: rll_description/urdf/egl90/egl90.xacro (robot description, xacro)
@@ -8,4 +8,5 @@
   <xacro:property name="joint_lower_limit" value="0.0" />
   <xacro:property name="joint_upper_limit" value="0.055" />
+  <xacro:property name="joint_damping" value="0.5" />
   <xacro:macro name="egl90" params="parent prefix">
     <joint name="gripper_adapter_joint" type="fixed">
@@ -58,4 +59,5 @@
       <axis xyz="1 0 0"/>
       <limit effort="500.0" lower="${joint_lower_limit}" upper="${joint_upper_limit}" velocity="0.1"/>
+      <dynamics damping="${joint_damping}"/>
     </joint>
     <link name="${prefix}gripper_waggon_left">
@@ -103,4 +105,5 @@
       <axis xyz="1 0 0"/>
       <limit effort="500.0" lower="${joint_lower_limit}" upper="${joint_upper_limit}" velocity="0.1"/>
+      <dynamics damping="${joint_damping}"/>
     </joint>
     <link name="${prefix}gripper_waggon_right">
